File: PCB/Sandy.kicad_pcb (KiCad board)
At the start: 2 copper layers, 285 x 95.1 mm, 249 parts, among them J1 USB_C_Receptacle_USB2.0, J2 Conn_01x03, J3 Conn_01x02, J5 Conn_02x03_Odd_Even, U1 ATmega32U4-MU, U2 24LC64, Y1 16MHz

Commit message: レイアウトテスト用としてスイッチを仮配置
Parts:
- removed D0, D1, D11, D12, D13, D14, D15, D16, D17, D18, D19, D2, D21, D22, D23, D24, D25, D26, D27, D28, D29, D3, D30, D31, D32, D33, D34, D35, D36, D37, D38, D39, D4, D40, D41, D42, D43, D44, D45, D46, D47, D48, D49, D5, D50, D51, D52, D53, D56, D57, D59, D6, D61, D62, D63, D64, D65, D67, D68, D69, D7, D71, D73, D74, D75, D78, D79, D8, D83, D84, D85, D87, D89, D9, D91, D92, D93, D94, D95, D96, D97, D98: D, Diode_SMD:D_SOD-123
- removed JP1: SolderJumper_2_Open, Jumper:SolderJumper-2_P1.3mm_Open_Pad1.0x1.5mm
- removed LED_STRIP1: Conn_01x03, locallib:LED_Strip
- removed LS1: Speaker, Buzzer_Beeper:Buzzer_Murata_PKMCS0909E4000-R1
- removed SW_'2, SW_LEFT1, SW_LWIN1u1, SW_[2, SW_]2, SW_narrow1u1, SW_narrowCTL1u1: SW_Push, MX_Alps_Hybrid:MXOnly-1U-Hotswap-guide
- removed SW_BS1.25u1, SW_ENT1.25u1, SW_ROPT1.25u1, SW_narrowRALT1.25u1: SW_Push, MX_Alps_Hybrid:MXOnly-1.25U-Hotswap-guide
- removed SW_BS1.25u2, SW_ENT1.25u2, SW_narrowRWIN1.25u1: SW_Push, MX_Alps_Hybrid:MXOnly-1.25U-Hotswap-guide-Rotate
- removed SW_BS1.5u2, SW_ENT1.5u2: SW_Push, MX_Alps_Hybrid:MXOnly-1.5U-Hotswap-guide-Rotate
- removed SW_BS2u1: SW_Push, MX_Alps_Hybrid:MXOnly-2U-Hotswap-guide
- removed SW_ENT2.25u1: SW_Push, MX_Alps_Hybrid:MXOnly-2.25U-Hotswap-LeftRotate-guide
- removed SW_LALT1.5u/MHEN1u1, SW_RALT1.5u1: SW_Push, MX_Alps_Hybrid:MXOnly-1.5U-Hotswap-guide
- removed SW_LSFT1.75u1: SW_Push, MX_Alps_Hybrid:MXOnly-1.75U-Hotswap-guide
- removed SW_LSPC2.25u1: SW_Push, MX_Alps_Hybrid:MXOnly-2.25U-Hotswap-guide
- added REF**: 1.75U, MX_Alps_Hybrid:MXOnly-1.75U-NoLED, F.Cu at (43.7, 88.9)
- added REF**: 2U, MX_Alps_Hybrid:MXOnly-2U-Hotswap, F.Cu at (41.3, 88.9)
- added REF**: 1.25U, MX_Alps_Hybrid:MXOnly-1.25U-NoLED, F.Cu at (38.9, 50.8)
- added SW_RALT1.25u1: SW_Push, MX_Alps_Hybrid:MXOnly-1.25U-Hotswap-guide, F.Cu at (258.0, 108.0)
- moved JP_LED1 68.2 mm to (42.0, 126.8)
- moved J2 51.4 mm to (242.8, 125.8)
- moved JP_LED2 50.7 mm to (228.2, 125.8)
- moved J5 50.6 mm to (102.2, 124.8)
- moved SW_LSFT2u1 48.6 mm to (-6.33, 98.5), turned to 0 degrees
- turned SW_L1 to 0 degrees
- turned SW_O1 to 0 degrees
Routing:
- net GND: track 571.7 -> 0.00 mm, vias 16 -> 0
- net +5V: track 499.2 -> 0.00 mm, vias 20 -> 0
- net MISO: track 378.9 -> 0.00 mm, vias 4 -> 0
- net MOSI: track 349.9 -> 0.00 mm, vias 6 -> 0
- net pin4: track 320.2 -> 0.00 mm, vias 1 -> 0
- net pin5: track 308.6 -> 0.00 mm, vias 3 -> 0
- net SCK: track 306.5 -> 0.00 mm, vias 5 -> 0
- net pin3: track 296.3 -> 0.00 mm, vias 4 -> 0
- net RE2_1: track 294.4 -> 0.00 mm, vias 8 -> 0
- net pin9: track 291.2 -> 0.00 mm, vias 4 -> 0
- net pin2: track 286.6 -> 0.00 mm, vias 3 -> 0
- net pin7: track 285.6 -> 0.00 mm, vias 3 -> 0
- net RE1_1: track 263.7 -> 0.00 mm, vias 7 -> 0
- net pin8: track 256.6 -> 0.00 mm, vias 4 -> 0
- net Net-(D42-Pad1): track 251.4 -> 0.00 mm, vias 6 -> 0
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- removed copper zone on B.Cu, net GND
- removed copper zone on F.Cu, net GND
Other:
- board text added: "#Sandy_kbd v.0, a cosmopolitan's keyboard by @jpskenn"
- board text added: "LED"
- board text added: "ResetSW"
- board text removed: "#Jones_kbd v.1.01 (042), a cosmopolitan's keyboard by @jpskenn"

Commit message: 基板重ね合わせのテスト
Parts:
- removed SW_CSPC2u1: SW_Push, MX_Alps_Hybrid:MXOnly-2U-Hotswap-ReversedStabilizers-guide
- added REF**: PinSocket_2x03_P2.54mm_Vertical_Dual_Entry, Jones.local:PinSocket_2x03_P2.54mm_Vertical_Dual_Entry, F.Cu at (271.2, 34.8)

Commit message: 子基板との接続を仮作成
Parts:
- removed LOGO1: #Jones_kbd v.1 (042), locallib:Jones_logo_B_R_60x98.2
- removed the REF** at (271.2, 34.8)
- removed SW_LSFT2u1: SW_Push, MX_Alps_Hybrid:MXOnly-2U-Hotswap-ReversedStabilizers-guide
- added REF**: PinHeader_2x02_P2.54mm_Vertical, Connector_PinHeader_2.54mm:PinHeader_2x02_P2.54mm_Vertical, F.Cu at (34.2, 23.4)
- added REF**: 1U, Jones.local:MXOnly-1U-Hotswap-guide-dummy, F.Cu at (137.7, 22.3)
- added REF**: 1U, Jones.local:MXOnly-1U-Hotswap-guide-dummy, F.Cu at (175.8, 79.4)
- added REF**: 1U, Jones.local:MXOnly-1U-Hotswap-guide-dummy, F.Cu at (156.8, 22.3)
- added REF**: 1U, Jones.local:MXOnly-1U-Hotswap-guide-dummy, F.Cu at (52.0, 41.3)
- added REF**: 1U, Jones.local:MXOnly-1U-Hotswap-guide-dummy, F.Cu at (156.8, 79.4)
- added REF**: 1U, Jones.local:MXOnly-1U-Hotswap-guide-dummy, F.Cu at (109.2, 41.3)
- added REF**: PinHeader_2x02_P2.54mm_Vertical, Connector_PinHeader_2.54mm:PinHeader_2x02_P2.54mm_Vertical, F.Cu at (110.4, 23.4)
- added REF**: 1U, Jones.local:MXOnly-1U-Hotswap-guide-dummy, F.Cu at (213.9, 22.3)
- added REF**: 1U, Jones.local:MXOnly-1U-Hotswap-guide-dummy, F.Cu at (290.1, 22.3)
- added REF**: PinHeader_2x02_P2.54mm_Vertical, Connector_PinHeader_2.54mm:PinHeader_2x02_P2.54mm_Vertical, F.Cu at (205.6, 23.4)
- added REF**: PinHeader_2x04_P2.54mm_Vertical, Connector_PinHeader_2.54mm:PinHeader_2x04_P2.54mm_Vertical, F.Cu at (19.6, 29.3)
- added REF**: PinHeader_1x04_P2.54mm_Vertical, Connector_PinHeader_2.54mm:PinHeader_1x04_P2.54mm_Vertical, F.Cu at (133.9, 68.7)
- added REF**: 1U, Jones.local:MXOnly-1U-Hotswap-guide-dummy, F.Cu at (147.3, 41.3)
- added REF**: 1U, Jones.local:MXOnly-1U-Hotswap-guide-dummy, F.Cu at (61.5, 22.3)
- added REF**: PinHeader_2x04_P2.54mm_Vertical, Connector_PinHeader_2.54mm:PinHeader_2x04_P2.54mm_Vertical, F.Cu at (114.9, 29.4)
- added REF**: 1U, Jones.local:MXOnly-1U-Hotswap-guide-dummy, F.Cu at (185.4, 60.4)
- added REF**: 1U, Jones.local:MXOnly-1U-Hotswap-guide-dummy, F.Cu at (166.3, 41.3)
- added REF**: 1U, Jones.local:MXOnly-1U-Hotswap-guide-dummy, F.Cu at (28.2, 41.3)
- added REF**: 1U, Jones.local:MXOnly-1U-Hotswap-guide-dummy, F.Cu at (252.0, 22.3)
- added REF**: 1U, Jones.local:MXOnly-1U-Hotswap-guide-dummy, F.Cu at (42.5, 22.3)
- added REF**: 1U, Jones.local:MXOnly-1U-Hotswap-guide-dummy, F.Cu at (23.4, 22.3)
- added REF**: PinHeader_1x04_P2.54mm_Vertical, Connector_PinHeader_2.54mm:PinHeader_1x04_P2.54mm_Vertical, F.Cu at (172.0, 68.7)
- added REF**: 1U, Jones.local:MXOnly-1U-Hotswap-guide-dummy, F.Cu at (194.9, 22.3)
- added REF**: PinHeader_1x04_P2.54mm_Vertical, Connector_PinHeader_2.54mm:PinHeader_1x04_P2.54mm_Vertical, F.Cu at (172.0, 49.6)
- added REF**: 1U, Jones.local:MXOnly-1U-Hotswap-guide-dummy, F.Cu at (118.7, 22.3)
- added REF**: 1U, Jones.local:MXOnly-1U-Hotswap-guide-dummy, F.Cu at (233.0, 22.3)
- added REF**: 1U, Jones.local:MXOnly-1U-Hotswap-guide-dummy, F.Cu at (80.6, 22.3)
- added REF**: 1U, Jones.local:MXOnly-1U-Hotswap-guide-dummy, F.Cu at (271.1, 22.3)
- added REF**: 1U, Jones.local:MXOnly-1U-Hotswap-guide-dummy, F.Cu at (137.7, 79.4)
- added REF**: 1U, Jones.local:MXOnly-1U-Hotswap-guide-dummy, F.Cu at (261.6, 41.3)
- added REF**: 1U, Jones.local:MXOnly-1U-Hotswap-guide-dummy, F.Cu at (147.3, 60.4)
- added REF**: 1U, Jones.local:MXOnly-1U-Hotswap-guide-dummy, F.Cu at (175.8, 22.3)
- added REF**: 1U, Jones.local:MXOnly-1U-Hotswap-guide-dummy, F.Cu at (204.4, 41.3)
- added REF**: 1U, Jones.local:MXOnly-1U-Hotswap-guide-dummy, F.Cu at (128.2, 41.3)
- added REF**: 1U, Jones.local:MXOnly-1U-Hotswap-guide-dummy, F.Cu at (99.6, 22.3)
- added REF**: PinHeader_2x04_P2.54mm_Vertical, Connector_PinHeader_2.54mm:PinHeader_2x04_P2.54mm_Vertical, F.Cu at (286.4, 29.3)
- added REF**: 1U, Jones.local:MXOnly-1U-Hotswap-guide-dummy, F.Cu at (285.4, 41.3)
- added REF**: 1U, Jones.local:MXOnly-1U-Hotswap-guide-dummy, F.Cu at (166.3, 60.4)
- added REF**: 1U, Jones.local:MXOnly-1U-Hotswap-guide-dummy, F.Cu at (185.4, 41.3)
- added REF**: 1U, Jones.local:MXOnly-1U-Hotswap-guide-dummy, F.Cu at (128.2, 60.4)
- added REF**: PinHeader_2x02_P2.54mm_Vertical, Connector_PinHeader_2.54mm:PinHeader_2x02_P2.54mm_Vertical, F.Cu at (281.8, 23.4)
- added REF**: PinHeader_2x04_P2.54mm_Vertical, Connector_PinHeader_2.54mm:PinHeader_2x04_P2.54mm_Vertical, F.Cu at (191.1, 29.3)
- added REF**: PinHeader_1x04_P2.54mm_Vertical, Connector_PinHeader_2.54mm:PinHeader_1x04_P2.54mm_Vertical, F.Cu at (133.9, 49.6)
- moved SW_7 112.2 mm to (194.9, 143.7)
- moved SW_-1 112.2 mm to (271.1, 143.7)
- moved SW_0 112.2 mm to (252.0, 143.7)
- moved SW_1 112.2 mm to (42.5, 143.7), turned to 0 degrees
- moved SW_2 112.2 mm to (61.5, 143.7)
- moved SW_3 112.2 mm to (80.6, 143.7)
- moved SW_4 112.2 mm to (99.6, 143.7)
- moved SW_5 112.2 mm to (118.7, 143.7)
- moved SW_6 112.2 mm to (137.7, 143.7)
- moved SW_8 112.2 mm to (213.9, 143.7)
- moved SW_9 112.2 mm to (233.0, 143.7)
- moved SW_=1 112.2 mm to (290.1, 143.7)
- moved SW_ESC1 112.2 mm to (23.4, 143.7), turned to 0 degrees
- moved SW_\1 112.2 mm to (175.8, 143.7)
- moved SW_`1 112.2 mm to (156.8, 143.7)
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Other:
- board text added: "to Mid"
- board text added: "to Top"

Commit message: MCUさっくり配置
Parts:
- moved C2 54.7 mm to (50.7, 17.8), turned to 180 degrees
- moved C4 53.2 mm to (59.0, 23.5), turned to 0 degrees
- moved Y1 49.3 mm to (50.6, 21.9), turned to -90 degrees
- moved C3 46.3 mm to (47.0, 22.8), turned to 90 degrees
- moved C7 38.3 mm to (44.1, 27.8), turned to -90 degrees
- moved U1 38.0 mm to (52.8, 32.2), turned to 0 degrees
- moved R6 34.8 mm to (58.6, 42.3), turned to 90 degrees
- moved C5 32.3 mm to (56.5, 42.3), turned to 90 degrees
- moved C6 31.9 mm to (41.2, 31.8), turned to -90 degrees
- moved C1 23.8 mm to (47.3, 40.6), turned to 180 degrees
- moved R5 21.6 mm to (47.3, 42.8), turned to 0 degrees
- moved D10 17.1 mm to (24.3, 21.0)
- moved F1 6.64 mm to (41.3, 17.5)
- moved R3 6.47 mm to (39.8, 23.3), turned to 180 degrees
- moved R4 4.54 mm to (39.7, 21.2), turned to 180 degrees
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
Commit message: 子基板仮配置。コネクタ形状、位置を変更。
Parts:
- removed the REF** at (133.9, 68.7)
- removed the REF** at (172.0, 68.7)
- removed the REF** at (172.0, 49.6)
- removed the REF** at (133.9, 49.6)
- added REF**: PinHeader_2x02_P2.54mm_Vertical, Connector_PinHeader_2.54mm:PinHeader_2x02_P2.54mm_Vertical, F.Cu at (174.6, 67.4)
- added REF**: PinHeader_2x02_P2.54mm_Vertical, Connector_PinHeader_2.54mm:PinHeader_2x02_P2.54mm_Vertical, F.Cu at (136.5, 46.0)
- added REF**: 60_Outline, locallib:60_Outline-Sandy-Top-NoSwImage, F.Cu at (156.8, 60.3)
- added REF**: PinHeader_2x02_P2.54mm_Vertical, Connector_PinHeader_2.54mm:PinHeader_2x02_P2.54mm_Vertical, F.Cu at (174.6, 46.0)
- added REF**: 60_Outline, locallib:60_Outline-Sandy-Mid-NoSwImage, F.Cu at (156.8, 60.3)
- added REF**: PinHeader_2x02_P2.54mm_Vertical, Connector_PinHeader_2.54mm:PinHeader_2x02_P2.54mm_Vertical, F.Cu at (136.5, 67.4)
