File: PCB/Sandy.kicad_pcb (KiCad board)
At the start: 2 copper layers, 285 x 95.1 mm, 189 parts, among them J1 USB_C_Receptacle_USB2.0, J2 Conn_01x03, J3 Conn_01x02, J5 Conn_02x03_Odd_Even, U1 ATmega32U4-MU, U2 24LC64, Y1 16MHz

Commit message: Base基板、中央、右下ネジ穴を大穴へ。issue_#23
Parts:
- added REF**: 1.25U, MX_Alps_Hybrid:MXOnly-1.25U-NoLED, F.Cu at (30.2, 41.3)
- REF**: footprint locallib:60_Outline-TinyHole_No_Hole3_WithNarrowFrame -> locallib:60_Outline-TinyHole_No_Hole3_Less_Hole
- REF**: footprint locallib:60_Outline-Sandy-Top-NoSwImage -> locallib:60_Outline-Sandy-Top-NoSwImage-WithHole
- REF**: footprint locallib:60_Outline-Sandy-Mid-NoSwImage -> locallib:60_Outline-Sandy-Mid-NoSwImage-WithHole
- turned SW_Z1 to 0 degrees
Other:
- outline, holes or cut-outs redrawn

Commit message: 外形、ネジ穴調整
Parts:
- removed the REF** at (34.2, 23.4)
- removed the REF** at (30.2, 41.3)
- added G***: LOGO, locallib:Jones_logo_B_8.3x13.9, B.Cu at (18.6, 36.5)
- added REF**: PinSocket_2x02_P2.54mm_Vertical_Duel_Entry, Connector_PinSocket_2.54mm:PinSocket_2x02_P2.54mm_Vertical_Duel_Entry, F.Cu at (31.7, 25.2)
- added REF**: MountingHole_5.3mm_M5, MountingHole:MountingHole_5.3mm_M5, F.Cu at (39.5, 40.9)
- REF**: footprint locallib:60_Outline-TinyHole_No_Hole3_Less_Hole -> locallib:60_Outline-TinyHole_No_Hole3_Less_Hole2
- REF** (x4): value PinHeader_2x04_P2.54mm_Vertical -> PinHeader_2x02_P2.54mm_Vertical; footprint Connector_PinHeader_2.54mm:PinHeader_2x04_P2.54mm_Vertical -> Connector_PinHeader_2.54mm:PinHeader_2x02_P2.54mm_Vertical
- REF**: footprint locallib:60_Outline-Sandy-Top-NoSwImage-WithHole -> locallib:60_Outline-Sandy-Top-NoSwImage-WithHole2
- REF**: footprint locallib:60_Outline-Sandy-Mid-NoSwImage-WithHole -> locallib:60_Outline-Sandy-Mid-NoSwImage-WithHole2
- moved REF** 6.65 mm to (117.4, 23.2), turned to 0 degrees
- moved REF** 6.49 mm to (193.6, 23.4), turned to 0 degrees
- moved REF** 6.43 mm to (22.2, 23.2), turned to 0 degrees
- moved REF** 6.35 mm to (288.9, 23.2), turned to 0 degrees
- moved REF** 2.55 mm to (107.9, 23.2), turned to 0 degrees
- moved REF** 2.47 mm to (279.3, 23.2), turned to 0 degrees
- moved REF** 2.47 mm to (203.1, 23.2), turned to 0 degrees
- moved REF** 1.30 mm to (136.5, 44.7)
- moved REF** 1.30 mm to (174.6, 44.7)
- moved REF** 1.27 mm to (174.6, 68.7)
- moved REF** 1.01 mm to (136.5, 68.4)
Other:
- outline, holes or cut-outs redrawn
- board text added: "#Jones_kbd Keyplate v.4.0.2, @jpskenn"

Commit message: キースイッチを配置
Parts:
- removed EXT_DP2, EXT_DP6: Conn_01x01, TestPoint:TestPoint_THTPad_D1.5mm_Drill0.7mm
- removed R7: 1k, Resistor_SMD:R_0805_2012Metric_Pad1.15x1.40mm_HandSolder
- removed the REF** at (174.6, 68.7)
- removed the REF** at (31.7, 25.2)
- removed the REF** at (136.5, 44.7)
- removed the REF** at (107.9, 23.2)
- removed the REF** at (203.1, 23.2)
- removed the REF** at (22.2, 23.2)
- removed the REF** at (117.4, 23.2)
- removed the REF** at (35.3, 79.4)
- removed the REF** at (33.0, 79.4)
- removed the REF** at (30.6, 162.7)
- removed the REF** at (174.6, 44.7)
- removed the REF** at (288.9, 23.2)
- removed the REF** at (136.5, 68.4)
- removed the REF** at (279.3, 23.2)
- removed the REF** at (193.6, 23.4)
- removed Reserve_AUDIO1, Reserve_AUDIO2, Reserve_PB5, Reserve_PC7, Reserve_PD5, Reserve_PF0, Reserve_PF6, Reserve_PF7: Conn_01x01, TestPoint:TestPoint_THTPad_D1.0mm_Drill0.5mm
- removed SW_0, SW_B1, SW_B2, SW_Center1: SW_Push, MX_Alps_Hybrid:MXOnly-1U-Hotswap-guide
- removed the SW_;1 at (147.3, 181.8)
- removed the SW_RALT1.25u1 at (249.7, 98.5)
- removed SW_RE1, SW_RE2: Rotary_Encoder_Switch, locallib:RotaryEncoder_Alps_EC11K-Switch_Vertical_H20mm
- added D1: D, Diode_SMD:D_SOD-123, F.Cu at (191.4, 176.3)
- added D11: D, Diode_SMD:D_SOD-123, F.Cu at (110.2, 194.0)
- added D12: D, Diode_SMD:D_SOD-123, F.Cu at (179.9, 176.3)
- added D13: D, Diode_SMD:D_SOD-123, F.Cu at (216.2, 173.6)
- added D14: D, Diode_SMD:D_SOD-123, F.Cu at (197.1, 176.3)
- added D15: D, Diode_SMD:D_SOD-123, F.Cu at (239.2, 209.1)
- added D16: D, Diode_SMD:D_SOD-123, F.Cu at (224.5, 156.9)
- added D17: D, Diode_SMD:D_SOD-123, F.Cu at (205.5, 159.6)
- added D18: D, Diode_SMD:D_SOD-123, F.Cu at (152.1, 175.5)
- added D19: D, Diode_SMD:D_SOD-123, F.Cu at (224.5, 153.6)
- added D2: D, Diode_SMD:D_SOD-123, F.Cu at (284.2, 160.6)
- added D20: D, Diode_SMD:D_SOD-123, F.Cu at (194.0, 159.6)
- added D21: D, Diode_SMD:D_SOD-123, F.Cu at (131.9, 202.4)
- added D22: D, Diode_SMD:D_SOD-123, F.Cu at (126.8, 178.1)
- added D23: D, Diode_SMD:D_SOD-123, F.Cu at (188.2, 159.6)
- added D24: D, Diode_SMD:D_SOD-123, F.Cu at (78.4, 161.3)
- added D25: D, Diode_SMD:D_SOD-123, F.Cu at (199.7, 159.6)
- added D26: D, Diode_SMD:D_SOD-123, F.Cu at (218.8, 156.9)
- added D27: D, Diode_SMD:D_SOD-123, F.Cu at (104.5, 199.0)
- added D28: D, Diode_SMD:D_SOD-123, F.Cu at (84.2, 154.6)
- added D29: D, Diode_SMD:D_SOD-123, F.Cu at (182.5, 159.6)
- added D3: D, Diode_SMD:D_SOD-123, F.Cu at (284.5, 154.6)
- added D30: D, Diode_SMD:D_SOD-123, F.Cu at (157.8, 175.5)
- added D31: D, Diode_SMD:D_SOD-123, F.Cu at (137.6, 195.7)
- added D32: D, Diode_SMD:D_SOD-123, F.Cu at (98.7, 195.6)
- added D33: D, Diode_SMD:D_SOD-123, F.Cu at (152.1, 178.8)
- added D34: D, Diode_SMD:D_SOD-123, F.Cu at (85.9, 209.8)
- added D35: D, Diode_SMD:D_SOD-123, F.Cu at (73.8, 221.9)
- added D36: D, Diode_SMD:D_SOD-123, F.Cu at (131.9, 199.0)
- added D37: D, Diode_SMD:D_SOD-123, F.Cu at (120.1, 184.6)
- added D38: D, Diode_SMD:D_SOD-123, F.Cu at (73.8, 228.6)
- added D39: D, Diode_SMD:D_SOD-123, F.Cu at (85.6, 216.5)
- added D4: D, Diode_SMD:D_SOD-123, F.Cu at (216.2, 170.3)
- added D40: D, Diode_SMD:D_SOD-123, F.Cu at (132.9, 172.1)
- added D41: D, Diode_SMD:D_SOD-123, F.Cu at (79.5, 221.9)
- added D42: D, Diode_SMD:D_SOD-123, F.Cu at (131.9, 195.7)
- added D43: D, Diode_SMD:D_SOD-123, F.Cu at (78.4, 158.0)
- added D44: D, Diode_SMD:D_SOD-123, F.Cu at (79.5, 225.2)
- added D45: D, Diode_SMD:D_SOD-123, F.Cu at (78.4, 164.7)
- added D46: D, Diode_SMD:D_SOD-123, F.Cu at (98.7, 199.0)
- added D47: D, Diode_SMD:D_SOD-123, F.Cu at (78.4, 154.6)
- added D48: D, Diode_SMD:D_SOD-123, F.Cu at (84.2, 151.3)
- added D49: D, Diode_SMD:D_SOD-123, F.Cu at (138.0, 163.8)
- added D5: D, Diode_SMD:D_SOD-123, F.Cu at (278.5, 164.0)
- added D50: D, Diode_SMD:D_SOD-123, F.Cu at (217.0, 160.3)
- added D51: D, Diode_SMD:D_SOD-123, F.Cu at (110.5, 190.7)
- added D52: D, Diode_SMD:D_SOD-123, F.Cu at (104.8, 190.7)
- added D53: D, Diode_SMD:D_SOD-123, F.Cu at (114.3, 184.6)
- added D54: D, Diode_SMD:D_SOD-123, F.Cu at (222.7, 160.3)
- added D55: D, Diode_SMD:D_SOD-123, F.Cu at (211.2, 159.6)
- added D56: D, Diode_SMD:D_SOD-123, F.Cu at (126.8, 174.8)
- added D57: D, Diode_SMD:D_SOD-123, F.Cu at (132.9, 168.7)
- added D58: D, Diode_SMD:D_SOD-123, F.Cu at (218.8, 153.6)
- added D59: D, Diode_SMD:D_SOD-123, F.Cu at (73.8, 225.2)
- added D6: D, Diode_SMD:D_SOD-123, F.Cu at (185.6, 176.3)
- added D7: D, Diode_SMD:D_SOD-123, F.Cu at (278.5, 160.6)
- added D74: D, Diode_SMD:D_SOD-123, F.Cu at (98.7, 205.7)
- added D79: D, Diode_SMD:D_SOD-123, F.Cu at (91.6, 213.1)
- added D8: D, Diode_SMD:D_SOD-123, F.Cu at (202.9, 176.3)
- added D84: D, Diode_SMD:D_SOD-123, F.Cu at (79.8, 215.8)
- added D87: D, Diode_SMD:D_SOD-123, F.Cu at (78.4, 151.3)
- added D89: D, Diode_SMD:D_SOD-123, F.Cu at (156.5, 148.5)
- added D9: D, Diode_SMD:D_SOD-123, F.Cu at (208.6, 176.3)
- added D91: D, Diode_SMD:D_SOD-123, F.Cu at (143.7, 163.8)
- added D92: D, Diode_SMD:D_SOD-123, F.Cu at (98.7, 202.3)
- added D93: D, Diode_SMD:D_SOD-123, F.Cu at (91.6, 209.8)
- added D94: D, Diode_SMD:D_SOD-123, F.Cu at (85.9, 213.1)
- added D96: D, Diode_SMD:D_SOD-123, F.Cu at (104.5, 202.3)
- added D97: D, Diode_SMD:D_SOD-123, F.Cu at (104.5, 195.6)
- added D98: D, Diode_SMD:D_SOD-123, F.Cu at (84.2, 158.0)
- added EXT_C10: Conn_01x01, TestPoint:TestPoint_THTPad_D2.0mm_Drill1.0mm, F.Cu at (289.7, 148.9)
- added EXT_C11: Conn_01x01, TestPoint:TestPoint_THTPad_D2.0mm_Drill1.0mm, F.Cu at (289.1, 159.0)
- added EXT_C12: Conn_01x01, TestPoint:TestPoint_THTPad_D2.0mm_Drill1.0mm, F.Cu at (289.4, 154.9)
- added EXT_C13: Conn_01x01, TestPoint:TestPoint_THTPad_D2.0mm_Drill1.0mm, F.Cu at (221.1, 174.7)
- added EXT_C14: Conn_01x01, TestPoint:TestPoint_THTPad_D2.0mm_Drill1.0mm, F.Cu at (274.1, 175.1)
- added EXT_C15: Conn_01x01, TestPoint:TestPoint_THTPad_D2.0mm_Drill1.0mm, F.Cu at (258.6, 189.3)
- added EXT_C16: Conn_01x01, TestPoint:TestPoint_THTPad_D2.0mm_Drill1.0mm, F.Cu at (151.2, 186.6)
- added EXT_C17: Conn_01x01, TestPoint:TestPoint_THTPad_D2.0mm_Drill1.0mm, F.Cu at (136.8, 203.4)
- added EXT_C18: Conn_01x01, TestPoint:TestPoint_THTPad_D2.0mm_Drill1.0mm, F.Cu at (140.8, 200.1)
- added EXT_C19: Conn_01x01, TestPoint:TestPoint_THTPad_D2.0mm_Drill1.0mm, F.Cu at (162.7, 175.8)
- added EXT_C20: Conn_01x01, TestPoint:TestPoint_THTPad_D2.0mm_Drill1.0mm, F.Cu at (233.5, 153.9)
- added EXT_C21: Conn_01x01, TestPoint:TestPoint_THTPad_D2.0mm_Drill1.0mm, F.Cu at (151.2, 182.5)
- added EXT_C22: Conn_01x01, TestPoint:TestPoint_THTPad_D2.0mm_Drill1.0mm, F.Cu at (157.0, 179.2)
- added EXT_C23: Conn_01x01, TestPoint:TestPoint_THTPad_D2.0mm_Drill1.0mm, F.Cu at (142.5, 196.0)
- added EXT_C8: Conn_01x01, TestPoint:TestPoint_THTPad_D2.0mm_Drill1.0mm, F.Cu at (283.4, 164.3)
- added EXT_C9: Conn_01x01, TestPoint:TestPoint_THTPad_D2.0mm_Drill1.0mm, F.Cu at (213.5, 177.3)
- added EXT_R10: Conn_01x01, TestPoint:TestPoint_THTPad_D2.0mm_Drill1.0mm, F.Cu at (280.2, 168.4)
- added EXT_R11: Conn_01x01, TestPoint:TestPoint_THTPad_D2.0mm_Drill1.0mm, F.Cu at (268.1, 181.2)
- added EXT_R12: Conn_01x01, TestPoint:TestPoint_THTPad_D2.0mm_Drill1.0mm, F.Cu at (272.1, 181.2)
- added EXT_R13: Conn_01x01, TestPoint:TestPoint_THTPad_D2.0mm_Drill1.0mm, F.Cu at (244.1, 209.5)
- added EXT_R14: Conn_01x01, TestPoint:TestPoint_THTPad_D2.0mm_Drill1.0mm, F.Cu at (268.1, 185.2)
- added EXT_R15: Conn_01x01, TestPoint:TestPoint_THTPad_D2.0mm_Drill1.0mm, F.Cu at (238.4, 212.8)
- added EXT_R16: Conn_01x01, TestPoint:TestPoint_THTPad_D2.0mm_Drill1.0mm, F.Cu at (221.1, 170.6)
- added EXT_R17: Conn_01x01, TestPoint:TestPoint_THTPad_D2.0mm_Drill1.0mm, F.Cu at (225.1, 170.6)
- added EXT_R20: Conn_01x01, TestPoint:TestPoint_THTPad_D2.0mm_Drill1.0mm, F.Cu at (131.0, 206.1)
- added EXT_R21: Conn_01x01, TestPoint:TestPoint_THTPad_D2.0mm_Drill1.0mm, F.Cu at (229.4, 153.9)
- added EXT_R22: Conn_01x01, TestPoint:TestPoint_THTPad_D2.0mm_Drill1.0mm, F.Cu at (136.8, 199.4)
- added EXT_R23: Conn_01x01, TestPoint:TestPoint_THTPad_D2.0mm_Drill1.0mm, F.Cu at (229.4, 158.0)
- added J10: Conn_02x02_Top_Bottom, Connector_PinHeader_2.00mm:PinHeader_2x02_P2.00mm_Vertical, F.Cu at (209.3, 170.6)
- added J11: Conn_02x02_Top_Bottom, Connector_PinHeader_2.00mm:PinHeader_2x02_P2.00mm_Vertical, F.Cu at (97.9, 189.9)
- added J12: Conn_02x02_Top_Bottom, Connector_PinHeader_2.00mm:PinHeader_2x02_P2.00mm_Vertical, F.Cu at (203.2, 170.6)
- added J13: Conn_02x02_Top_Bottom, Connector_PinHeader_2.00mm:PinHeader_2x02_P2.00mm_Vertical, F.Cu at (107.4, 185.0)
- added J14: Conn_02x02_Top_Bottom, Connector_PinHeader_2.00mm:PinHeader_2x02_P2.00mm_Vertical, F.Cu at (277.6, 154.9)
- added J15: Conn_02x02_Top_Bottom, Connector_PinHeader_2.00mm:PinHeader_2x02_P2.00mm_Vertical, F.Cu at (268.1, 169.1)
- added J16: Conn_02x02_Top_Bottom, Connector_PinHeader_2.00mm:PinHeader_2x02_P2.00mm_Vertical, F.Cu at (197.2, 170.6)
- added J17: Conn_02x02_Top_Bottom, Connector_PinHeader_2.00mm:PinHeader_2x02_P2.00mm_Vertical, F.Cu at (277.6, 148.9)
- added J18: Conn_02x02_Top_Bottom, Connector_PinHeader_2.00mm:PinHeader_2x02_P2.00mm_Vertical, F.Cu at (179.0, 170.6)
- added J19: Conn_02x02_Top_Bottom, Connector_PinHeader_2.00mm:PinHeader_2x02_P2.00mm_Vertical, F.Cu at (185.1, 170.6)
- added J20: Conn_02x02_Top_Bottom, Connector_PinHeader_2.00mm:PinHeader_2x02_P2.00mm_Vertical, F.Cu at (268.1, 175.1)
- added J21: Conn_02x02_Top_Bottom, Connector_PinHeader_2.00mm:PinHeader_2x02_P2.00mm_Vertical, F.Cu at (205.8, 153.9)
- added J22: Conn_02x02_Top_Bottom, Connector_PinHeader_2.00mm:PinHeader_2x02_P2.00mm_Vertical, F.Cu at (181.6, 153.9)
- added J23: Conn_02x02_Top_Bottom, Connector_PinHeader_2.00mm:PinHeader_2x02_P2.00mm_Vertical, F.Cu at (187.7, 153.9)
- added J24: Conn_02x02_Top_Bottom, Connector_PinHeader_2.00mm:PinHeader_2x02_P2.00mm_Vertical, F.Cu at (211.9, 153.9)
- added J25: Conn_02x02_Top_Bottom, Connector_PinHeader_2.00mm:PinHeader_2x02_P2.00mm_Vertical, F.Cu at (274.1, 169.1)
- added J26: Conn_02x02_Top_Bottom, Connector_PinHeader_2.00mm:PinHeader_2x02_P2.00mm_Vertical, F.Cu at (283.7, 148.9)
- added J27: Conn_02x02_Top_Bottom, Connector_PinHeader_2.00mm:PinHeader_2x02_P2.00mm_Vertical, F.Cu at (193.7, 153.9)
- added J28: Conn_02x02_Top_Bottom, Connector_PinHeader_2.00mm:PinHeader_2x02_P2.00mm_Vertical, F.Cu at (199.8, 153.9)
- added J5: Conn_02x02_Top_Bottom, Connector_PinHeader_2.00mm:PinHeader_2x02_P2.00mm_Vertical, F.Cu at (79.0, 210.1)
- added J6: Conn_02x02_Top_Bottom, Connector_PinHeader_2.00mm:PinHeader_2x02_P2.00mm_Vertical, F.Cu at (72.9, 210.1)
- added J7: Conn_02x02_Top_Bottom, Connector_PinHeader_2.00mm:PinHeader_2x02_P2.00mm_Vertical, F.Cu at (126.0, 169.1)
- added J8: Conn_02x02_Top_Bottom, Connector_PinHeader_2.00mm:PinHeader_2x02_P2.00mm_Vertical, F.Cu at (72.9, 216.2)
- added J9: Conn_02x02_Top_Bottom, Connector_PinHeader_2.00mm:PinHeader_2x02_P2.00mm_Vertical, F.Cu at (191.1, 170.6)
- added LOGO1: #Sandy_kbd v.0, locallib:Jones_logo_B_R_60x98.2, F.Cu at (-70.6, -92.0)
- added REF**: 60_Outline, locallib:60_Outline-Sandy-Mid-NoSwImage-WithHole2, F.Cu at (156.8, -34.9)
- added REF**: 60_Outline, locallib:60_Outline-Sandy-Top-NoSwImage-WithHole2, F.Cu at (155.6, -83.7)
- added SW_10: SW_Push, MX_Alps_Hybrid:MXOnly-1U-Hotswap-guide, F.Cu at (250.8, -121.8)
- added SW_;3: SW_Push, MX_Alps_Hybrid:MXOnly-1U-NoLED, F.Cu at (147.3, -34.9)
- added SW_ENT1.25u1: SW_Push, MX_Alps_Hybrid:MXOnly-1.25U-Hotswap-guide, F.Cu at (283.0, 60.4)
- added SW_LSFT1.75u1: SW_Push, MX_Alps_Hybrid:MXOnly-1.75U-NoLED, F.Cu at (35.3, 79.4)
- added SW_LSFT2u1: SW_Push, MX_Alps_Hybrid:MXOnly-2U-Hotswap-guide, F.Cu at (33.0, 79.4)
- added SW_R4CenterC1: SW_Push, MX_Alps_Hybrid:MXOnly-1U-Hotswap-guide, F.Cu at (156.8, -15.8)
- added SW_R4CenterL1: SW_Push, MX_Alps_Hybrid:MXOnly-1U-Hotswap-guide, F.Cu at (137.7, -15.8)
- added SW_R4CenterR1: SW_Push, MX_Alps_Hybrid:MXOnly-1U-Hotswap-guide, F.Cu at (175.8, -15.8)
- added SW_RE_L1: RotaryEncoder_Switch, locallib:RotaryEncoder_Alps_EC11K-Switch_Vertical_H20mm, F.Cu at (137.1, 152.0)
- added SW_RE_L2: RotaryEncoder_Switch, locallib:RotaryEncoder_Alps_EC11K-Switch_Vertical_H20mm, F.Cu at (40.5, 154.7)
- added SW_RE_R1: RotaryEncoder_Switch, locallib:RotaryEncoder_Alps_EC11K-Switch_Vertical_H20mm, F.Cu at (107.4, 172.8)
- added SW_RE_R2: RotaryEncoder_Switch, locallib:RotaryEncoder_Alps_EC11K-Switch_Vertical_H20mm, F.Cu at (59.0, 154.7)
- added SW_ROPT1.25u1: SW_Push, MX_Alps_Hybrid:MXOnly-1.25U-Hotswap-guide, F.Cu at (249.7, 98.5)
- added SW_TAB1.25u1: SW_Push, MX_Alps_Hybrid:MXOnly-1.25U-NoLED, F.Cu at (30.6, -53.9)
- EXT_C0: renamed from EXT_DP9; footprint TestPoint:TestPoint_THTPad_D1.5mm_Drill0.7mm -> TestPoint:TestPoint_THTPad_D2.0mm_Drill1.0mm
- EXT_C1: renamed from EXT_DP8; footprint TestPoint:TestPoint_THTPad_D1.5mm_Drill0.7mm -> TestPoint:TestPoint_THTPad_D2.0mm_Drill1.0mm
- EXT_C2: renamed from EXT_DP4; footprint TestPoint:TestPoint_THTPad_D1.5mm_Drill0.7mm -> TestPoint:TestPoint_THTPad_D2.0mm_Drill1.0mm
- EXT_C3: renamed from EXT_DP0; footprint TestPoint:TestPoint_THTPad_D1.5mm_Drill0.7mm -> TestPoint:TestPoint_THTPad_D2.0mm_Drill1.0mm
- EXT_C4: renamed from EXT_DP5; footprint TestPoint:TestPoint_THTPad_D1.5mm_Drill0.7mm -> TestPoint:TestPoint_THTPad_D2.0mm_Drill1.0mm
- EXT_C5: renamed from EXT_DP3; footprint TestPoint:TestPoint_THTPad_D1.5mm_Drill0.7mm -> TestPoint:TestPoint_THTPad_D2.0mm_Drill1.0mm
- EXT_C6: renamed from EXT_DP7; footprint TestPoint:TestPoint_THTPad_D1.5mm_Drill0.7mm -> TestPoint:TestPoint_THTPad_D2.0mm_Drill1.0mm
- EXT_C7: renamed from EXT_DP1; footprint TestPoint:TestPoint_THTPad_D1.5mm_Drill0.7mm -> TestPoint:TestPoint_THTPad_D2.0mm_Drill1.0mm
- EXT_R0: renamed from EXT_P0; footprint TestPoint:TestPoint_THTPad_D1.5mm_Drill0.7mm -> TestPoint:TestPoint_THTPad_D2.0mm_Drill1.0mm
- EXT_R1: renamed from EXT_P1; footprint TestPoint:TestPoint_THTPad_D1.5mm_Drill0.7mm -> TestPoint:TestPoint_THTPad_D2.0mm_Drill1.0mm
- EXT_R2: renamed from EXT_P2; footprint TestPoint:TestPoint_THTPad_D1.5mm_Drill0.7mm -> TestPoint:TestPoint_THTPad_D2.0mm_Drill1.0mm
- EXT_R3: renamed from EXT_P3; footprint TestPoint:TestPoint_THTPad_D1.5mm_Drill0.7mm -> TestPoint:TestPoint_THTPad_D2.0mm_Drill1.0mm
- EXT_R4: renamed from EXT_P4; footprint TestPoint:TestPoint_THTPad_D1.5mm_Drill0.7mm -> TestPoint:TestPoint_THTPad_D2.0mm_Drill1.0mm
- EXT_R5: renamed from EXT_P5; footprint TestPoint:TestPoint_THTPad_D1.5mm_Drill0.7mm -> TestPoint:TestPoint_THTPad_D2.0mm_Drill1.0mm
- EXT_R6: renamed from EXT_P6; footprint TestPoint:TestPoint_THTPad_D1.5mm_Drill0.7mm -> TestPoint:TestPoint_THTPad_D2.0mm_Drill1.0mm
- EXT_R7: renamed from EXT_P7; footprint TestPoint:TestPoint_THTPad_D1.5mm_Drill0.7mm -> TestPoint:TestPoint_THTPad_D2.0mm_Drill1.0mm
- EXT_R8: renamed from EXT_P8; footprint TestPoint:TestPoint_THTPad_D1.5mm_Drill0.7mm -> TestPoint:TestPoint_THTPad_D2.0mm_Drill1.0mm
- EXT_R9: renamed from EXT_P9; footprint TestPoint:TestPoint_THTPad_D1.5mm_Drill0.7mm -> TestPoint:TestPoint_THTPad_D2.0mm_Drill1.0mm
- SW_;2: footprint MX_Alps_Hybrid:MXOnly-1U-NoLED -> MX_Alps_Hybrid:MXOnly-1U-Hotswap-guide
- moved G*** 346.8 mm to (-324.1, -16.4)
- moved REF** 346.8 mm to (-303.3, -12.0)
- moved SW_6 268.1 mm to (174.6, -121.8)
- moved SW_\1 266.3 mm to (155.6, -121.8)
- moved SW_`1 266.3 mm to (136.5, -121.8)
- moved SW_7 265.5 mm to (193.7, -121.8)
- moved SW_9 265.5 mm to (231.8, -121.8)
- moved SW_8 265.5 mm to (212.7, -121.8)
- moved SW_1 265.5 mm to (41.3, -121.8)
- moved SW_2 265.5 mm to (60.3, -121.8)
- moved SW_3 265.5 mm to (79.4, -121.8)
- moved SW_4 265.5 mm to (98.4, -121.8)
- moved SW_5 265.5 mm to (117.5, -121.8)
- moved SW_ESC1 265.5 mm to (22.2, -121.8)
- moved SW_=1 265.5 mm to (288.9, -121.8)
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- renumbered J5 to J4, SW_;3 to SW_;1
Connections:
- EXT_C0 pad 1: RE2_1 -> RE_L1_1
- EXT_C1 pad 1: Net-(D8-Pad1) -> SCK
- EXT_C2 pad 1: Net-(D7-Pad1) -> MOSI
- EXT_C3 pad 1: Net-(D6-Pad1) -> MISO
- EXT_C4 pad 1: Net-(D4-Pad1) -> RE_R2_1
- EXT_C5 pad 1: Net-(D42-Pad1) -> col5
- EXT_C6 pad 1: Net-(D2-Pad1) -> col6
- EXT_C7 pad 1: RE1_1 -> RE_R1_1
- EXT_R0 pad 1: MISO -> row0
- EXT_R1 pad 1: MOSI -> row1
- EXT_R2 pad 1: pin2 -> row2
- EXT_R3 pad 1: pin3 -> row3
- EXT_R4 pad 1: pin4 -> row4
- EXT_R5 pad 1: pin5 -> row5
- EXT_R6 pad 1: SCK -> row6
- EXT_R7 pad 1: pin7 -> row7
- EXT_R8 pad 1: pin8 -> row8
- EXT_R9 pad 1: pin9 -> row9
- J1 pad A8: (no net) -> unconnected-(J1-PadA8)
- J1 pad B8: (no net) -> unconnected-(J1-PadB8)
- SW_'1 pad 1: Net-(D5-Pad1) -> Mid_col3
- SW_-1 pad 1: RE1_1 -> Top_col6
- SW_1 pad 1: RE2_1 -> Top_col0
- SW_2 pad 1: Net-(D8-Pad1) -> Top_col1
- SW_3 pad 1: Net-(D7-Pad1) -> Top_col1
- SW_4 pad 1: Net-(D7-Pad1) -> Top_col2
- SW_5 pad 1: Net-(D6-Pad1) -> Top_col2
- SW_6 pad 1: Net-(D5-Pad1) -> Top_col3
- SW_7 pad 1: Net-(D3-Pad1) -> Top_col4
- SW_8 pad 1: Net-(D3-Pad1) -> Top_col5
- SW_9 pad 1: Net-(D42-Pad1) -> Top_col5
- SW_;1 pad 1: Net-(D2-Pad1) -> col6
- SW_;2 pad 1: Net-(D6-Pad1) -> Mid_col3
- SW_<1 pad 1: Net-(D42-Pad1) -> col5
- SW_=1 pad 1: RE1_1 -> Top_col7
- SW_>1 pad 1: Net-(D2-Pad1) -> col6
- SW_A1 pad 1: RE2_1 -> RE_L1_1
- SW_BS1.5u1 pad 1: RE1_1 -> Mid_col6
- SW_C1 pad 1: Net-(D7-Pad1) -> MOSI
- SW_CAPS1u1 pad 1: RE2_1 -> RE_L1_1
- SW_CAPS1u1 pad 2: RE2_2 -> RE_L1_2
- SW_CTL1.25u1 pad 1: RE2_1 -> RE_L1_1
- SW_CTL1.5u1 pad 1: RE2_1 -> RE_L1_1
- SW_CenterL1u1 pad 1: Net-(D5-Pad1) -> MISO
- SW_CenterL1u1 pad 2: Net-(D22-Pad2) -> RE_L2_2
- SW_CenterR1u1 pad 1: Net-(D4-Pad1) -> RE_R2_1
- SW_CenterR1u1 pad 2: Net-(D40-Pad2) -> RE_R2_2
- SW_D1 pad 1: Net-(D7-Pad1) -> SCK
- SW_DOWN1 pad 1: RE1_1 -> col6
- SW_E1 pad 1: Net-(D7-Pad1) -> SCK
- SW_ENT1.5u1 pad 1: RE1_1 -> col6
- SW_ESC1 pad 1: RE2_1 -> Top_col0
- SW_F1 pad 1: Net-(D7-Pad1) -> MOSI
- SW_Fn1u1 pad 1: RE1_1 -> RE_R1_1
- SW_G1 pad 1: Net-(D6-Pad1) -> Mid_col2
- SW_H1 pad 1: Net-(D4-Pad1) -> Mid_col4
- SW_I1 pad 1: Net-(D3-Pad1) -> col5
- SW_J1 pad 1: Net-(D3-Pad1) -> RE_R2_1
- SW_K1 pad 1: Net-(D42-Pad1) -> col5
- SW_L1 pad 1: Net-(D42-Pad1) -> col5
- SW_L2-1u1 pad 1: Net-(D8-Pad1) -> RE_L1_1
- SW_LALT1.25u1 pad 1: Net-(D7-Pad1) -> SCK
- SW_LSFT1u1 pad 1: RE2_1 -> RE_L1_1
- SW_LSFT1u2 pad 1: RE2_1 -> RE_L1_1
- SW_LSPC2u1 pad 1: Net-(D6-Pad1) -> MOSI
- SW_LWIN1.25u1 pad 1: Net-(D8-Pad1) -> SCK
- SW_M1 pad 1: Net-(D3-Pad1) -> col5
- SW_N1 pad 1: Net-(D3-Pad1) -> RE_R2_1
- SW_O1 pad 1: Net-(D42-Pad1) -> col5
- SW_P1 pad 1: Net-(D2-Pad1) -> Mid_col6
- SW_Q1 pad 1: RE2_1 -> Mid_col0
- SW_R1 pad 1: Net-(D7-Pad1) -> Mid_col2
- SW_RALT1.25u1 pad 1: Net-(D42-Pad1) -> col5
- SW_RIGHT1 pad 1: RE1_1 -> RE_R1_1
- SW_RIGHT1 pad 2: RE1_2 -> RE_R1_2
- SW_RSPC2u1 pad 1: Net-(D3-Pad1) -> RE_R2_1
- SW_S1 pad 1: Net-(D8-Pad1) -> SCK
- SW_T1 pad 1: Net-(D6-Pad1) -> Top_col2
- SW_TAB1.5u1 pad 1: RE2_1 -> Mid_col0
- SW_U1 pad 1: Net-(D3-Pad1) -> Mid_col4
- SW_UP1 pad 1: RE1_1 -> col6
- SW_V1 pad 1: Net-(D6-Pad1) -> MOSI
- SW_W1 pad 1: Net-(D8-Pad1) -> SCK
- SW_X1 pad 1: Net-(D7-Pad1) -> SCK
- SW_Y1 pad 1: Net-(D4-Pad1) -> Top_col4
- SW_Z1 pad 1: Net-(D8-Pad1) -> SCK
- SW_[1 pad 1: Net-(D6-Pad1) -> Top_col3
- SW_\1 pad 1: Net-(D4-Pad1) -> Top_col4
- SW_]1 pad 1: Net-(D5-Pad1) -> Top_col3
- SW_`1 pad 1: Net-(D5-Pad1) -> Top_col3
- U1 pad 1: pin2 -> row6
- U1 pad 12: pin7 -> RE_R1_1
- U1 pad 20: RE1_A -> RE_L_A
- U1 pad 21: RE1_B -> RE_L_B
- U1 pad 22: resv_PD5 -> row3
- U1 pad 25: pin4 -> row2
- U1 pad 26: pin3 -> row4
- U1 pad 27: pin9 -> row5
- U1 pad 28: pin8 -> RE_R2_1
- U1 pad 29: resv_PB5 -> col5
- U1 pad 30: AUDIO2 -> col6
- U1 pad 31: AUDIO1 -> row0
- U1 pad 32: resv_PC7 -> row1
- U1 pad 36: resv_PF7 -> row9
- U1 pad 37: resv_PF6 -> row8
- U1 pad 38: RE2_A -> RE_R_A
- U1 pad 39: RE2_B -> RE_R_B
- U1 pad 41: resv_PF0 -> row7
- U1 pad 42: (no net) -> unconnected-(U1-Pad42)
- U1 pad 8: pin5 -> RE_L1_1
Other:
- board size 285 x 95.1 mm -> 626.8 x 112.9 mm

Commit message: 部品仮配置
Parts:
- removed the J15 at (268.1, 169.1)
- removed the J17 at (277.6, 148.9)
- removed the J25 at (274.1, 169.1)
- removed the J26 at (283.7, 148.9)
- added J17 (x2): Conn_02x02_Top_Bottom, locallib:PinHeader_2x02_P2.00mm_Vertical_Centered, F.Cu at (33.0, -62.3)
- added J18: Conn_02x02_Top_Bottom, locallib:PinHeader_2x02_P2.00mm_Vertical_Centered, F.Cu at (109.2, -62.1)
- added J21: Conn_02x02_Top_Bottom, locallib:PinHeader_2x02_P2.00mm_Vertical_Centered, F.Cu at (137.7, -38.5)
- added J22: Conn_02x02_Top_Bottom, locallib:PinHeader_2x02_P2.00mm_Vertical_Centered, F.Cu at (175.8, -38.5)
- J10: renamed from J13; footprint Connector_PinHeader_2.00mm:PinHeader_2x02_P2.00mm_Vertical -> locallib:PinHeader_2x02_P2.00mm_Vertical_Centered
- J11: renamed from J9; footprint Connector_PinHeader_2.00mm:PinHeader_2x02_P2.00mm_Vertical -> locallib:PinHeader_2x02_P2.00mm_Vertical_Centered
- J12: renamed from J10; footprint Connector_PinHeader_2.00mm:PinHeader_2x02_P2.00mm_Vertical -> locallib:PinHeader_2x02_P2.00mm_Vertical_Centered
- J13: renamed from J12; footprint Connector_PinHeader_2.00mm:PinHeader_2x02_P2.00mm_Vertical -> locallib:PinHeader_2x02_P2.00mm_Vertical_Centered
- J14, J19, J20, J27, J28, J5, J6, J7, J8: footprint Connector_PinHeader_2.00mm:PinHeader_2x02_P2.00mm_Vertical -> locallib:PinHeader_2x02_P2.00mm_Vertical_Centered
- J15: renamed from J16; footprint Connector_PinHeader_2.00mm:PinHeader_2x02_P2.00mm_Vertical -> locallib:PinHeader_2x02_P2.00mm_Vertical_Centered
- J16: renamed from J18; footprint Connector_PinHeader_2.00mm:PinHeader_2x02_P2.00mm_Vertical -> locallib:PinHeader_2x02_P2.00mm_Vertical_Centered
- J23: renamed from J21; footprint Connector_PinHeader_2.00mm:PinHeader_2x02_P2.00mm_Vertical -> locallib:PinHeader_2x02_P2.00mm_Vertical_Centered
- J24: renamed from J22; footprint Connector_PinHeader_2.00mm:PinHeader_2x02_P2.00mm_Vertical -> locallib:PinHeader_2x02_P2.00mm_Vertical_Centered
- J25: renamed from J23; footprint Connector_PinHeader_2.00mm:PinHeader_2x02_P2.00mm_Vertical -> locallib:PinHeader_2x02_P2.00mm_Vertical_Centered
- J26: renamed from J24; footprint Connector_PinHeader_2.00mm:PinHeader_2x02_P2.00mm_Vertical -> locallib:PinHeader_2x02_P2.00mm_Vertical_Centered
- J9: renamed from J11; footprint Connector_PinHeader_2.00mm:PinHeader_2x02_P2.00mm_Vertical -> locallib:PinHeader_2x02_P2.00mm_Vertical_Centered
- SW_CAPS1u1, SW_CenterL1u1, SW_CenterR1u1, SW_RIGHT1: footprint MX_Alps_Hybrid:MXOnly-1U-Hotswap-guide -> MX_Alps_Hybrid:MXOnly-1U-Hotswap-on-RE-guide
- SW_RE_L1, SW_RE_L2, SW_RE_R1, SW_RE_R2: footprint locallib:RotaryEncoder_Alps_EC11K-Switch_Vertical_H20mm -> locallib:RotaryEncoder_Alps_EC11K-Switch_Vertical_H20mm_NPTH_MP
- moved D21 349.0 mm to (237.8, -130.2)
- moved D36 349.0 mm to (237.8, -133.5)
- moved D31 349.0 mm to (243.5, -136.9)
- moved D42 349.0 mm to (237.8, -136.9)
- moved EXT_TC1 348.9 mm to (163.7, -144.4)
- moved EXT_TC7 347.2 mm to (210.4, -144.4)
- moved EXT_TC2 345.9 mm to (171.1, -144.4)
- moved EXT_TR0 343.7 mm to (144.9, -137.3)
- moved EXT_TC0 331.1 mm to (155.6, -144.4)
- moved EXT_TC5 329.9 mm to (194.9, -144.4)
- moved EXT_TR1 328.5 mm to (144.9, -129.0)
- moved D18 327.5 mm to (227.2, -143.3)
- moved D30 327.5 mm to (233.0, -143.3)
- moved D33 327.5 mm to (227.2, -139.9)
- moved EXT_TC6 326.8 mm to (202.0, -144.4)
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- renumbered EXT_C8 to EXT_MC0, EXT_C9 to EXT_MC1, EXT_C10 to EXT_MC2, EXT_C11 to EXT_MC3, EXT_C12 to EXT_MC4, EXT_C13 to EXT_MC5, EXT_C14 to EXT_MC6, EXT_C15 to EXT_MC7, EXT_R10 to EXT_MR0, EXT_R12 to EXT_MR1, EXT_R14 to EXT_MR2, EXT_R16 to EXT_MR3, EXT_R11 to EXT_MR5, EXT_R13 to EXT_MR6, EXT_R15 to EXT_MR7, EXT_R17 to EXT_MR8, EXT_C16 to EXT_TC0, EXT_C17 to EXT_TC1, EXT_C18 to EXT_TC2, EXT_C19 to EXT_TC3, EXT_C20 to EXT_TC4, EXT_C21 to EXT_TC5, EXT_C22 to EXT_TC6, EXT_C23 to EXT_TC7, EXT_R20 to EXT_TR0, EXT_R22 to EXT_TR1, EXT_R21 to EXT_TR5, EXT_R23 to EXT_TR6
Other:
- board text added: "to Base"

Commit message: スイッチ方向確定。細かな調整
Parts:
- removed the J17 at (33.0, -62.3) (x2)
- removed SW_;3: SW_Push, MX_Alps_Hybrid:MXOnly-1U-NoLED
- added J17: Conn_02x02_Top_Bottom, locallib:PinHeader_2x02_P2.00mm_Vertical_Centered, F.Cu at (33.0, -62.3)
- REF**: footprint locallib:60_Outline-Sandy-Top-NoSwImage-WithHole2 -> locallib:60_Outline-Sandy-Top-NoSwImage-WithHole2-ECO1
- REF**: footprint locallib:60_Outline-Sandy-Mid-NoSwImage-WithHole2 -> locallib:60_Outline-Sandy-Mid-NoSwImage-WithHole2-ECO1
- moved JP_LED2 146.5 mm to (73.4, 116.3)
- moved JP_LED1 31.5 mm to (65.1, 116.3)
- moved REF** 28.6 mm to (156.8, 31.8)
- moved REF** 9.50 mm to (156.8, 50.8)
- moved J24 0.16 mm to (109.2, -110.6)
- moved J18 0.15 mm to (109.2, -62.3)
- turned SW_;2 to 0 degrees

Commit message: 5wayスイッチを追加するテスト
Parts:
- added REF**: SW_JS5208_add_MP_hole, locallib:SW_JS5208_add_MP_hole, F.Cu at (137.7, -6.32)
- added REF**: SW_JS5208_add_MP_hole, locallib:SW_JS5208_add_MP_hole, F.Cu at (175.8, -6.32)
- moved J4 116.7 mm to (54.3, 5.50)
- turned U1 to -90 degrees
Other:
- outline, holes or cut-outs redrawn

Commit message: JSTコネクタとスペーサーでなんとするテスト
Parts:
- removed the REF** at (137.7, -6.32)
- removed the REF** at (175.8, -6.32)
- added D60: D, Diode_SMD:D_SOD-123, F.Cu at (231.8, -5.13)
- added D61: D, Diode_SMD:D_SOD-123, F.Cu at (231.8, 1.57)
- added D62: D, Diode_SMD:D_SOD-123, F.Cu at (237.5, -5.13)
- added D63: D, Diode_SMD:D_SOD-123, F.Cu at (231.8, -1.78)
- added D64: D, Diode_SMD:D_SOD-123, F.Cu at (237.5, -1.78)
- added REF**: MountingHole_2.2mm_M2_No_Cu, MountingHole:MountingHole_2.2mm_M2_No_Cu, F.Cu at (17.5, -69.4)
- added REF**: JST_SH_SM04B-SRSS-TB_1x04-1MP_P1.00mm_Horizontal, Connector_JST:JST_SH_SM04B-SRSS-TB_1x04-1MP_P1.00mm_Horizontal, F.Cu at (41.3, -38.5)
- added REF**: JST_SH_SM04B-SRSS-TB_1x04-1MP_P1.00mm_Horizontal, Connector_JST:JST_SH_SM04B-SRSS-TB_1x04-1MP_P1.00mm_Horizontal, F.Cu at (272.3, 66.3)
- added REF**: JST_SH_SM04B-SRSS-TB_1x04-1MP_P1.00mm_Horizontal, Connector_JST:JST_SH_SM04B-SRSS-TB_1x04-1MP_P1.00mm_Horizontal, F.Cu at (273.5, -38.5)
- added REF**: MountingHole_2.2mm_M2_No_Cu, MountingHole:MountingHole_2.2mm_M2_No_Cu, F.Cu at (17.5, -38.5)
- added REF**: MountingHole_2.2mm_M2_No_Cu, MountingHole:MountingHole_2.2mm_M2_No_Cu, F.Cu at (17.4, -118.2)
- added REF**: JST_SH_SM04B-SRSS-TB_1x04-1MP_P1.00mm_Horizontal, Connector_JST:JST_SH_SM04B-SRSS-TB_1x04-1MP_P1.00mm_Horizontal, F.Cu at (41.3, 66.3)
- added REF**: JST_SH_SM04B-SRSS-TB_1x04-1MP_P1.00mm_Horizontal, Connector_JST:JST_SH_SM04B-SRSS-TB_1x04-1MP_P1.00mm_Horizontal, F.Cu at (273.5, -50.4)
- added REF**: JST_SH_SM04B-SRSS-TB_1x04-1MP_P1.00mm_Horizontal, Connector_JST:JST_SH_SM04B-SRSS-TB_1x04-1MP_P1.00mm_Horizontal, F.Cu at (80.1, 50.8)
- added REF**: JST_SH_SM04B-SRSS-TB_1x04-1MP_P1.00mm_Horizontal, Connector_JST:JST_SH_SM04B-SRSS-TB_1x04-1MP_P1.00mm_Horizontal, F.Cu at (233.5, 50.8)
- added S1: JS5208, locallib:SW_JS5208_add_MP_hole, F.Cu at (137.7, -6.33)
- added S2: JS5208, locallib:SW_JS5208_add_MP_hole, F.Cu at (175.8, -6.33)

Commit message: JSTコネクタとスペーサーに置き換え
Parts:
- removed J10, J15, J16, J20, J21, J22, J26, J27, J28, J9: Conn_02x02_Top_Bottom, locallib:PinHeader_2x02_P2.00mm_Vertical_Centered
- removed the REF** at (17.5, -69.4)
- removed the REF** at (41.3, -38.5)
- removed the REF** at (272.3, 66.3)
- removed the REF** at (273.5, -38.5)
- removed the REF** at (17.5, -38.5)
- removed the REF** at (17.4, -118.2)
- removed the REF** at (41.3, 66.3)
- removed the REF** at (273.5, -50.4)
- removed the REF** at (80.1, 50.8)
- removed the REF** at (233.5, 50.8)
- added H10: MountingHole, MountingHole:MountingHole_2.2mm_M2_No_Cu, F.Cu at (296.1, 47.3)
- added H11: MountingHole, MountingHole:MountingHole_2.2mm_M2_No_Cu, F.Cu at (17.5, 47.3)
- added H12: MountingHole, MountingHole:MountingHole_2.2mm_M2_No_Cu, F.Cu at (296.1, 15.9)
- added H13: MountingHole, MountingHole:MountingHole_2.2mm_M2_No_Cu, F.Cu at (137.7, 69.9)
- added H14: MountingHole, MountingHole:MountingHole_2.2mm_M2_No_Cu, F.Cu at (175.8, 69.9)
- added H15: MountingHole, MountingHole:MountingHole_2.2mm_M2_No_Cu, F.Cu at (17.5, -69.8)
- added H16: MountingHole, MountingHole:MountingHole_2.2mm_M2_No_Cu, F.Cu at (90.1, -63.5)
- added H17: MountingHole, MountingHole:MountingHole_2.2mm_M2_No_Cu, F.Cu at (156.8, -63.5)
- added H18: MountingHole, MountingHole:MountingHole_2.2mm_M2_No_Cu, F.Cu at (223.5, -63.5)
- added H19: MountingHole, MountingHole:MountingHole_2.2mm_M2_No_Cu, F.Cu at (296.1, -69.4)
- added H20: MountingHole, MountingHole:MountingHole_2.2mm_M2_No_Cu, F.Cu at (17.5, -38.5)
- added H21: MountingHole, MountingHole:MountingHole_2.2mm_M2_No_Cu, F.Cu at (296.1, -38.5)
- added H22: MountingHole, MountingHole:MountingHole_2.2mm_M2_No_Cu, F.Cu at (137.7, -15.9)
- added H23: MountingHole, MountingHole:MountingHole_2.2mm_M2_No_Cu, F.Cu at (175.8, -15.8)
- added H24: MountingHole, MountingHole:MountingHole_2.2mm_M2_No_Cu, F.Cu at (129.4, -69.9)
- added H25: MountingHole, MountingHole:MountingHole_2.2mm_M2_No_Cu, F.Cu at (186.6, -69.9)
- added H26: MountingHole, MountingHole:MountingHole_2.2mm_M2_No_Cu, F.Cu at (33.0, -61.6)
- added H27: MountingHole, MountingHole:MountingHole_2.2mm_M2_No_Cu, F.Cu at (71.1, -61.6)
- added H28: MountingHole, MountingHole:MountingHole_2.2mm_M2_No_Cu, F.Cu at (242.5, -61.6)
- added H29: MountingHole, MountingHole:MountingHole_2.2mm_M2_No_Cu, F.Cu at (280.6, -61.6)
- added H30: MountingHole, MountingHole:MountingHole_2.2mm_M2_No_Cu, F.Cu at (137.7, -39.0)
- added H31: MountingHole, MountingHole:MountingHole_2.2mm_M2_No_Cu, F.Cu at (175.8, -39.0)
- added H32: MountingHole, MountingHole:MountingHole_2.2mm_M2_No_Cu, F.Cu at (129.4, -118.2)
- added H33: MountingHole, MountingHole:MountingHole_2.2mm_M2_No_Cu, F.Cu at (186.6, -118.2)
- added H34: MountingHole, MountingHole:MountingHole_2.2mm_M2_No_Cu, F.Cu at (33.0, -109.9)
- added H35: MountingHole, MountingHole:MountingHole_2.2mm_M2_No_Cu, F.Cu at (71.1, -109.9)
- added H36: MountingHole, MountingHole:MountingHole_2.2mm_M2_No_Cu, F.Cu at (242.5, -109.9)
- added H37: MountingHole, MountingHole:MountingHole_2.2mm_M2_No_Cu, F.Cu at (280.6, -109.9)
- added H38: MountingHole, MountingHole:MountingHole_2.2mm_M2_No_Cu, F.Cu at (137.7, -87.3)
- added H39: MountingHole, MountingHole:MountingHole_2.2mm_M2_No_Cu, F.Cu at (175.8, -87.3)
- added H6: MountingHole, MountingHole:MountingHole_2.2mm_M2_No_Cu, F.Cu at (17.5, 15.9)
- added H7: MountingHole, MountingHole:MountingHole_2.2mm_M2_No_Cu, F.Cu at (90.1, 22.3)
- added H8: MountingHole, MountingHole:MountingHole_2.2mm_M2_No_Cu, F.Cu at (156.8, 22.3)
- added H9: MountingHole, MountingHole:MountingHole_2.2mm_M2_No_Cu, F.Cu at (223.5, 22.3)
- H1, H2, H3, H4, H5: footprint MountingHole:MountingHole_2.2mm_M2 -> MountingHole:MountingHole_2.2mm_M2_No_Cu
- J11, J12, J13, J14, J17, J18, J19, J23, J24, J25, J5, J6, J7, J8: footprint locallib:PinHeader_2x02_P2.00mm_Vertical_Centered -> Connector_JST:JST_SH_SM04B-SRSS-TB_1x04-1MP_P1.00mm_Horizontal
- moved J24 14.6 mm to (104.4, -96.8)
- moved J23 13.8 mm to (33.0, -96.8)
- moved J17 10.2 mm to (42.5, -65.9)
Connections:
- J17 pad 2: Mid_col0 -> Mid_row1
- J17 pad 4: Mid_col1 -> Mid_row6
- J23 pad 2: Top_col0 -> Top_row1
- J23 pad 4: Top_col1 -> Top_row6
