File: PCB/Sandy.kicad_pcb (KiCad board)
At the start: 2 copper layers, 626.8 x 112.9 mm, 326 parts, among them J1 USB_C_Receptacle_USB2.0, J11 Conn_02x02_Top_Bottom, J12 Conn_02x02_Top_Bottom, J13 Conn_02x02_Top_Bottom, J14 Conn_02x02_Top_Bottom, J17 Conn_02x02_Top_Bottom, J18 Conn_02x02_Top_Bottom, J19 Conn_02x02_Top_Bottom, J2 Conn_01x03, J23 Conn_02x02_Top_Bottom, J24 Conn_02x02_Top_Bottom, J25 Conn_02x02_Top_Bottom, J3 Conn_01x02, J4 Conn_02x03_Odd_Even, J5 Conn_02x02_Top_Bottom, J6 Conn_02x02_Top_Bottom, J7 Conn_02x02_Top_Bottom, J8 Conn_02x02_Top_Bottom, U1 ATmega32U4-MU, U2 24LC64, Y1 16MHz

Commit message: スペーサー位置調整
Parts:
- moved J8 134.1 mm to (156.8, 41.3), turned to 90 degrees
- moved J5 104.9 mm to (128.2, 33.0), turned to 90 degrees
- moved J7 38.6 mm to (156.8, 33.0), turned to 90 degrees
- moved J6 17.1 mm to (128.2, 41.3), turned to 90 degrees
- moved H17 6.45 mm to (156.8, -69.9)
- moved H8 6.44 mm to (156.8, 15.8)
- moved H16 1.89 mm to (90.1, -61.6)
- moved H7 1.89 mm to (90.1, 24.1)
- moved H9 1.89 mm to (223.5, 24.1)
- moved H18 1.88 mm to (223.5, -61.6)

Commit message: コネクタ位置考え中
Parts:
- added J10: Conn_01x04, Connector_PinHeader_2.54mm:PinHeader_1x04_P2.54mm_Vertical, F.Cu at (154.4, 35.1)
- added J15: Conn_01x04, Connector_PinHeader_2.54mm:PinHeader_1x04_P2.54mm_Vertical, F.Cu at (159.3, 20.8)
- added J16: Conn_01x04, Connector_PinHeader_2.54mm:PinHeader_1x04_P2.54mm_Vertical, F.Cu at (159.3, 35.1)
- added J20: Conn_01x04, Connector_PinHeader_2.54mm:PinHeader_1x04_P2.54mm_Vertical, F.Cu at (357.5, -50.2)
- added J21: Conn_01x04, Connector_PinHeader_2.54mm:PinHeader_1x04_P2.54mm_Vertical, F.Cu at (334.2, -50.2)
- added J22: Conn_01x04, Connector_PinHeader_2.54mm:PinHeader_1x04_P2.54mm_Vertical, F.Cu at (352.8, -50.2)
- added J26: Conn_01x04, Connector_PinHeader_2.54mm:PinHeader_1x04_P2.54mm_Vertical, F.Cu at (362.1, -50.2)
- added J27: Conn_01x04, Connector_PinHeader_2.54mm:PinHeader_1x04_P2.54mm_Vertical, F.Cu at (338.9, -50.2)
- added J28: Conn_01x04, Connector_PinHeader_2.54mm:PinHeader_1x04_P2.54mm_Vertical, F.Cu at (343.5, -50.2)
- added J29: Conn_01x04, Connector_PinHeader_2.54mm:PinHeader_1x04_P2.54mm_Vertical, F.Cu at (348.2, -50.2)
- added J30: Conn_01x04, Connector_PinHeader_2.54mm:PinHeader_1x04_P2.54mm_Vertical, F.Cu at (183.0, -160.1)
- added J31: Conn_01x04, Connector_PinHeader_2.54mm:PinHeader_1x04_P2.54mm_Vertical, F.Cu at (178.3, -160.1)
- added J32: Conn_01x04, Connector_PinHeader_2.54mm:PinHeader_1x04_P2.54mm_Vertical, F.Cu at (173.7, -160.1)
- added J9: Conn_01x04, Connector_PinHeader_2.54mm:PinHeader_1x04_P2.54mm_Vertical, F.Cu at (154.4, 20.8)
- J11, J12, J13, J14, J23, J24, J25: footprint Connector_JST:JST_SH_SM04B-SRSS-TB_1x04-1MP_P1.00mm_Horizontal -> locallib:JST_SH_BM04B-SRSS-TB_1x04-1MP_P1.00mm_Vertical_wCable_housing; moved to B.Cu
- J17, J18, J19, J5, J6, J7, J8: footprint Connector_JST:JST_SH_SM04B-SRSS-TB_1x04-1MP_P1.00mm_Horizontal -> locallib:JST_SH_BM04B-SRSS-TB_1x04-1MP_P1.00mm_Vertical_wCable_housing
- REF**: footprint locallib:60_Outline-Sandy-Mid-NoSwImage-WithHole2 -> locallib:60_Outline-Sandy-Mid-WithHole
- moved D13 132.9 mm to (392.5, -32.5)
- moved D2 132.9 mm to (347.3, -27.8)
- moved D4 132.9 mm to (392.5, -35.9)
- moved D5 132.9 mm to (341.5, -24.4)
- moved D60 132.9 mm to (364.0, -19.4)
- moved D61 132.9 mm to (364.0, -12.7)
- moved D62 132.9 mm to (369.7, -19.4)
- moved D63 132.9 mm to (364.0, -16.1)
- moved D64 132.9 mm to (369.7, -16.1)
- moved D7 132.9 mm to (341.5, -27.8)
- moved D1 132.9 mm to (367.7, -29.8)
- moved D12 132.9 mm to (356.2, -29.8)
- moved D14 132.9 mm to (373.5, -29.8)
- moved D15 132.9 mm to (348.5, -24.2)
- moved D3 132.9 mm to (347.6, -33.8)
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Other:
- board size 626.8 x 112.9 mm -> 626.8 x 136.3 mm
- board text added: "Topのコネクタ位置と、Midの穴を合わせるように、配置見直し。 TopとBaseのコネクタ位置がかぶらないように。 MidからTopへのコネクタを、Midうら面に配置したら？"

Commit message: 3枚の基板を1枚にまとめ中
Parts:
- removed G***: LOGO, locallib:Jones_logo_B_8.3x13.9
- removed H4: MountingHole, MountingHole:MountingHole_2.2mm_M2_No_Cu
- removed J16, J20, J21, J22, J26, J27, J28, J29, J30, J31, J32: Conn_01x04, Connector_PinHeader_2.54mm:PinHeader_1x04_P2.54mm_Vertical
- removed J17, J18, J19: Conn_02x02_Top_Bottom, locallib:JST_SH_BM04B-SRSS-TB_1x04-1MP_P1.00mm_Vertical_wCable_housing
- removed the REF** at (-303.3, -12.0)
- added H40: MountingHole, MountingHole:MountingHole_2.2mm_M2_No_Cu, F.Cu at (131.8, 69.9)
- added H41: MountingHole, MountingHole:MountingHole_2.2mm_M2_No_Cu, F.Cu at (181.8, 69.9)
- added H42: MountingHole, MountingHole:MountingHole_2.2mm_M2_No_Cu, B.Cu at (131.8, -15.8)
- added H43: MountingHole, MountingHole:MountingHole_2.2mm_M2_No_Cu, B.Cu at (181.8, -15.8)
- added REF**: 60_Outline, locallib:60_Outline-Sandy-Top-NoSwImage-WithHole2-ECO1, F.Cu at (156.8, -53.9)
- D1, D11, D12, D13, D14, D15, D16, D17, D18, D19, D2, D20, D21, D22, D23, D24, D25, D26, D27, D28, D29, D3, D30, D31, D32, D33, D34, D35, D36, D37, D38, D39, D4, D40, D41, D42, D43, D44, D45, D46, D47, D48, D49, D5, D50, D51, D52, D53, D54, D55, D56, D57, D58, D59, D6, D60, D61, D62, D63, D64, D7, D74, D79, D8, D84, D87, D89, D9, D91, D92, D93, D94, D96, D97, D98, EXT_MC0, EXT_MC1, EXT_MC2, EXT_MC3, EXT_MC4, EXT_MC5, EXT_MC6, EXT_MC7, EXT_MR0, EXT_MR1, EXT_MR2, EXT_MR3, EXT_MR5, EXT_MR6, EXT_MR7, EXT_MR8, EXT_TC0, EXT_TC1, EXT_TC2, EXT_TC3, EXT_TC4, EXT_TC5, EXT_TC6, EXT_TC7, EXT_TR0, EXT_TR1, EXT_TR5, EXT_TR6, H1, H15, H16, H17, H18, H19, H2, H20, H21, H22, H23, H3, H32, H33, H34, H35, H36, H37, H38, H39, H5: moved to B.Cu
- J10, J15, J9: value Conn_01x04 -> Conn_02x02_Top_Bottom; footprint Connector_PinHeader_2.54mm:PinHeader_1x04_P2.54mm_Vertical -> locallib:JST_SH_SM04B-SRSS-TB_1x04-1MP_P1.00mm_Horizontal_wCable_housing_spare_pin
- J11, J12, J13, J14, J23, J24, J25, J5, J6, J7, J8: footprint locallib:JST_SH_BM04B-SRSS-TB_1x04-1MP_P1.00mm_Vertical_wCable_housing -> locallib:JST_SH_SM04B-SRSS-TB_1x04-1MP_P1.00mm_Horizontal_wCable_housing_spare_pin
- REF**: footprint locallib:60_Outline-TinyHole_No_Hole3_Less_Hole2 -> locallib:60_Outline-Sandy-Base2
- REF**: footprint locallib:60_Outline-Sandy-Mid-WithHole -> locallib:60_Outline-Sandy-Mid-WithHole-wCutout2
- REF**: footprint locallib:60_Outline-Sandy-Top-NoSwImage-WithHole2 -> locallib:60_Outline-Sandy-Top-NoSwImage-WithHole3
- SW_LSFT2u1: footprint MX_Alps_Hybrid:MXOnly-2U-Hotswap-guide -> MX_Alps_Hybrid:MXOnly-2U-Hotswap-guide2
- SW_LSPC2u1, SW_RSPC2u1: footprint MX_Alps_Hybrid:MXOnly-2U-Hotswap-ReversedStabilizers-guide -> MX_Alps_Hybrid:MXOnly-2U-Hotswap-ReversedStabilizers-guide2
- moved D13 65.7 mm to (326.8, -33.7), turned to 180 degrees
- moved D4 65.7 mm to (326.8, -37.1), turned to 180 degrees
- moved EXT_TC7 65.5 mm to (148.5, -170.6), turned to 180 degrees
- moved EXT_TR0 65.5 mm to (213.9, -163.5), turned to 180 degrees
- moved EXT_TR1 65.5 mm to (213.9, -155.2), turned to 180 degrees
- moved EXT_MC0 59.5 mm to (384.2, -68.2), turned to 180 degrees
- moved EXT_MC7 59.5 mm to (324.7, -68.2), turned to 180 degrees
- moved D16 58.7 mm to (230.8, -159.7), turned to 180 degrees
- moved D19 58.7 mm to (230.8, -163.0), turned to 180 degrees
- moved D18 58.7 mm to (289.6, -169.4), turned to 180 degrees
- moved D33 58.7 mm to (289.6, -166.1), turned to 180 degrees
- moved D54 55.1 mm to (232.6, -156.3), turned to 180 degrees
- moved EXT_TR5 51.2 mm to (206.8, -161.1), turned to 180 degrees
- moved EXT_TR6 51.2 mm to (206.8, -154.0), turned to 180 degrees
- moved D9 50.6 mm to (334.4, -31.0), turned to 180 degrees
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Connections:
- J10 pad 1: row1 -> RE_L1_1
- J10 pad 3: row6 -> SCK
- J15 pad 1: row2 -> RE_R2_1
- J15 pad 2: RE_R2_1 -> col6
- J15 pad 3: row7 -> col5
- J15 pad 4: col5 -> RE_R1_1
- J9 pad 2: RE_L1_1 -> row1
- J9 pad 4: SCK -> row6
Other:
- board size 626.8 x 136.3 mm -> 285 x 95.1 mm
- board text removed: "#Jones_kbd Keyplate v.4.0.2, @jpskenn"
- board text removed: "2.75u"
