File: PCB/matrix_top.kicad_sch (KiCad schematic)
At the start: 61 parts, among them J23 Conn_02x02_Top_Bottom, J24 Conn_02x02_Top_Bottom, J25 Conn_02x02_Top_Bottom

Commit message: 基板外形置き換え
Parts:
- H32, H33, H34, H35, H36, H37, H38, H39: footprint MountingHole:MountingHole_2.2mm_M2_No_Cu -> MountingHole:MountingHole_2.2mm_M2_Pad; symbol Mechanical:MountingHole -> Mechanical:MountingHole_Pad
- SW_5, SW_8: footprint MX_Alps_Hybrid:MXOnly-1U-Hotswap-guide -> MX_Alps_Hybrid:MXOnly-1U-Hotswap-guide-screw-hole-side
Connections:
- new net Top_GND: H32.1, H33.1, H34.1, H35.1, H36.1, H37.1, H38.1, H39.1

Commit message: BaseからMidへのピン数減少のため、コネクタ1個減らす
Parts:
- H32, H33, H34, H35, H36, H37, H38, H39: footprint MountingHole:MountingHole_2.2mm_M2_Pad -> MountingHole:MountingHole_2.2mm_M2_Pad_minimal
Changed lines of the file:
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@@
       (effects (font (size 1.27 1.27)) (justify left))
     )
-    (property "Footprint" "MountingHole:MountingHole_2.2mm_M2_Pad" (id 2) (at 235.585 125.095 0)
+    (property "Footprint" "MountingHole:MountingHole_2.2mm_M2_Pad_minimal" (id 2) (at 235.585 125.095 0)
       (effects (font (size 1.27 1.27)) hide)
     )
@@
       (effects (font (size 1.27 1.27)) (justify left))
     )
-    (property "Footprint" "MountingHole:MountingHole_2.2mm_M2_Pad" (id 2) (at 271.145 131.445 0)
+    (property "Footprint" "MountingHole:MountingHole_2.2mm_M2_Pad_minimal" (id 2) (at 271.145 131.445 0)
       (effects (font (size 1.27 1.27)) hide)
     )
@@
       (effects (font (size 1.27 1.27)) (justify left))
     )
-    (property "Footprint" "MountingHole:MountingHole_2.2mm_M2_Pad" (id 2) (at 217.805 139.065 0)
+    (property "Footprint" "MountingHole:MountingHole_2.2mm_M2_Pad_minimal" (id 2) (at 217.805 139.065 0)
       (effects (font (size 1.27 1.27)) hide)
     )
@@
       (effects (font (size 1.27 1.27)) (justify left))
     )
-    (property "Footprint" "MountingHole:MountingHole_2.2mm_M2_Pad" (id 2) (at 235.585 139.065 0)
+    (property "Footprint" "MountingHole:MountingHole_2.2mm_M2_Pad_minimal" (id 2) (at 235.585 139.065 0)
       (effects (font (size 1.27 1.27)) hide)
     )
@@
       (effects (font (size 1.27 1.27)) (justify left))
     )
-    (property "Footprint" "MountingHole:MountingHole_2.2mm_M2_Pad" (id 2) (at 182.245 131.445 0)
+    (property "Footprint" "MountingHole:MountingHole_2.2mm_M2_Pad_minimal" (id 2) (at 182.245 131.445 0)
       (effects (font (size 1.27 1.27)) hide)
     )
@@
       (effects (font (size 1.27 1.27)) (justify left))
     )
-    (property "Footprint" "MountingHole:MountingHole_2.2mm_M2_Pad" (id 2) (at 200.025 131.445 0)
+    (property "Footprint" "MountingHole:MountingHole_2.2mm_M2_Pad_minimal" (id 2) (at 200.025 131.445 0)
       (effects (font (size 1.27 1.27)) hide)
     )
@@
       (effects (font (size 1.27 1.27)) (justify left))
     )
-    (property "Footprint" "MountingHole:MountingHole_2.2mm_M2_Pad" (id 2) (at 253.365 131.445 0)
+    (property "Footprint" "MountingHole:MountingHole_2.2mm_M2_Pad_minimal" (id 2) (at 253.365 131.445 0)
       (effects (font (size 1.27 1.27)) hide)
     )
@@
       (effects (font (size 1.27 1.27)) (justify left))
     )
-    (property "Footprint" "MountingHole:MountingHole_2.2mm_M2_Pad" (id 2) (at 217.805 125.095 0)
-      (effects (font (size 1.27 1.27)) hide)
-    )
+    (property "Footprint" "MountingHole:MountingHole_2.2mm_M2_Pad_minimal" (id 2) (at 217.805 125.095 0)
+      (effects (font (size 1.27 1.27)) hide)
+    )

Commit message: スイッチのソケットを廃止
Parts:
- SW_-1, SW_1, SW_10, SW_2, SW_3, SW_4, SW_6, SW_7, SW_9, SW_=1, SW_ESC1, SW_T1, SW_Y1, SW_[1, SW_\1, SW_]1, SW_`1: footprint MX_Alps_Hybrid:MXOnly-1U-Hotswap-guide -> MX_Alps_Hybrid:MXOnly-1U-NoLED
- SW_5, SW_8: footprint MX_Alps_Hybrid:MXOnly-1U-Hotswap-guide-screw-hole-side -> MX_Alps_Hybrid:MXOnly-1U-NoLED
Changed lines of the file:
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@@
     (property "Reference" "SW_8" (id 0) (at 208.28 51.181 0))
     (property "Value" "SW_Push" (id 1) (at 208.28 53.4924 0))
-    (property "Footprint" "MX_Alps_Hybrid:MXOnly-1U-Hotswap-guide-screw-hole-side" (id 2) (at 208.28 53.34 0)
+    (property "Footprint" "MX_Alps_Hybrid:MXOnly-1U-NoLED" (id 2) (at 208.28 53.34 0)
       (effects (font (size 1.27 1.27)) hide)
     )
@@
     (property "Reference" "SW_=1" (id 0) (at 274.32 51.181 0))
     (property "Value" "SW_Push" (id 1) (at 274.32 53.4924 0))
-    (property "Footprint" "MX_Alps_Hybrid:MXOnly-1U-Hotswap-guide" (id 2) (at 274.32 53.34 0)
+    (property "Footprint" "MX_Alps_Hybrid:MXOnly-1U-NoLED" (id 2) (at 274.32 53.34 0)
       (effects (font (size 1.27 1.27)) hide)
     )
@@
     (property "Reference" "SW_]1" (id 0) (at 158.75 82.931 0))
     (property "Value" "SW_Push" (id 1) (at 158.75 85.2424 0))
-    (property "Footprint" "MX_Alps_Hybrid:MXOnly-1U-Hotswap-guide" (id 2) (at 158.75 85.09 0)
+    (property "Footprint" "MX_Alps_Hybrid:MXOnly-1U-NoLED" (id 2) (at 158.75 85.09 0)
       (effects (font (size 1.27 1.27)) hide)
     )
@@
     (property "Reference" "SW_2" (id 0) (at 76.2 51.181 0))
     (property "Value" "SW_Push" (id 1) (at 76.2 53.4924 0))
-    (property "Footprint" "MX_Alps_Hybrid:MXOnly-1U-Hotswap-guide" (id 2) (at 76.2 53.34 0)
+    (property "Footprint" "MX_Alps_Hybrid:MXOnly-1U-NoLED" (id 2) (at 76.2 53.34 0)
       (effects (font (size 1.27 1.27)) hide)
     )
@@
     (property "Reference" "SW_T1" (id 0) (at 125.73 82.931 0))
     (property "Value" "SW_Push" (id 1) (at 125.73 85.2424 0))
-    (property "Footprint" "MX_Alps_Hybrid:MXOnly-1U-Hotswap-guide" (id 2) (at 125.73 85.09 0)
+    (property "Footprint" "MX_Alps_Hybrid:MXOnly-1U-NoLED" (id 2) (at 125.73 85.09 0)
       (effects (font (size 1.27 1.27)) hide)
     )
@@
     (property "Reference" "SW_6" (id 0) (at 142.24 51.181 0))
     (property "Value" "SW_Push" (id 1) (at 142.24 53.4924 0))
-    (property "Footprint" "MX_Alps_Hybrid:MXOnly-1U-Hotswap-guide" (id 2) (at 142.24 53.34 0)
+    (property "Footprint" "MX_Alps_Hybrid:MXOnly-1U-NoLED" (id 2) (at 142.24 53.34 0)
       (effects (font (size 1.27 1.27)) hide)
     )
@@
     (property "Reference" "SW_5" (id 0) (at 125.73 51.181 0))
     (property "Value" "SW_Push" (id 1) (at 125.73 53.4924 0))
-    (property "Footprint" "MX_Alps_Hybrid:MXOnly-1U-Hotswap-guide-screw-hole-side" (id 2) (at 125.73 53.34 0)
+    (property "Footprint" "MX_Alps_Hybrid:MXOnly-1U-NoLED" (id 2) (at 125.73 53.34 0)
       (effects (font (size 1.27 1.27)) hide)
     )
@@
     (property "Reference" "SW_Y1" (id 0) (at 175.26 82.931 0))
     (property "Value" "SW_Push" (id 1) (at 175.26 85.2424 0))
-    (property "Footprint" "MX_Alps_Hybrid:MXOnly-1U-Hotswap-guide" (id 2) (at 175.26 85.09 0)
+    (property "Footprint" "MX_Alps_Hybrid:MXOnly-1U-NoLED" (id 2) (at 175.26 85.09 0)
       (effects (font (size 1.27 1.27)) hide)
     )
@@
     (property "Reference" "SW_`1" (id 0) (at 158.75 51.181 0))
     (property "Value" "SW_Push" (id 1) (at 158.75 53.4924 0))
-    (property "Footprint" "MX_Alps_Hybrid:MXOnly-1U-Hotswap-guide" (id 2) (at 158.75 53.34 0)
+    (property "Footprint" "MX_Alps_Hybrid:MXOnly-1U-NoLED" (id 2) (at 158.75 53.34 0)
       (effects (font (size 1.27 1.27)) hide)
     )
@@
     (property "Reference" "SW_7" (id 0) (at 191.77 51.181 0))
     (property "Value" "SW_Push" (id 1) (at 191.77 53.4924 0))
-    (property "Footprint" "MX_Alps_Hybrid:MXOnly-1U-Hotswap-guide" (id 2) (at 191.77 53.34 0)
+    (property "Footprint" "MX_Alps_Hybrid:MXOnly-1U-NoLED" (id 2) (at 191.77 53.34 0)
       (effects (font (size 1.27 1.27)) hide)
     )
@@
     (property "Reference" "SW_9" (id 0) (at 224.79 51.181 0))
     (property "Value" "SW_Push" (id 1) (at 224.79 53.4924 0))
-    (property "Footprint" "MX_Alps_Hybrid:MXOnly-1U-Hotswap-guide" (id 2) (at 224.79 53.34 0)
+    (property "Footprint" "MX_Alps_Hybrid:MXOnly-1U-NoLED" (id 2) (at 224.79 53.34 0)
       (effects (font (size 1.27 1.27)) hide)
     )
@@
     (property "Reference" "SW_4" (id 0) (at 109.22 51.181 0))
     (property "Value" "SW_Push" (id 1) (at 109.22 53.4924 0))
-    (property "Footprint" "MX_Alps_Hybrid:MXOnly-1U-Hotswap-guide" (id 2) (at 109.22 53.34 0)
+    (property "Footprint" "MX_Alps_Hybrid:MXOnly-1U-NoLED" (id 2) (at 109.22 53.34 0)
       (effects (font (size 1.27 1.27)) hide)
     )
@@
     (property "Reference" "SW_3" (id 0) (at 92.71 51.181 0))
     (property "Value" "SW_Push" (id 1) (at 92.71 53.4924 0))
-    (property "Footprint" "MX_Alps_Hybrid:MXOnly-1U-Hotswap-guide" (id 2) (at 92.71 53.34 0)
+    (property "Footprint" "MX_Alps_Hybrid:MXOnly-1U-NoLED" (id 2) (at 92.71 53.34 0)
       (effects (font (size 1.27 1.27)) hide)
     )
@@
     (property "Reference" "SW_10" (id 0) (at 241.3 51.181 0))
     (property "Value" "SW_Push" (id 1) (at 241.3 53.4924 0))
-    (property "Footprint" "MX_Alps_Hybrid:MXOnly-1U-Hotswap-guide" (id 2) (at 241.3 53.34 0)
+    (property "Footprint" "MX_Alps_Hybrid:MXOnly-1U-NoLED" (id 2) (at 241.3 53.34 0)
       (effects (font (size 1.27 1.27)) hide)
     )
@@
     (property "Reference" "SW_ESC1" (id 0) (at 43.18 51.181 0))
     (property "Value" "SW_Push" (id 1) (at 43.18 53.4924 0))
-    (property "Footprint" "MX_Alps_Hybrid:MXOnly-1U-Hotswap-guide" (id 2) (at 43.18 53.34 0)
+    (property "Footprint" "MX_Alps_Hybrid:MXOnly-1U-NoLED" (id 2) (at 43.18 53.34 0)
       (effects (font (size 1.27 1.27)) hide)
     )
@@
     (property "Reference" "SW_-1" (id 0) (at 257.81 51.181 0))
     (property "Value" "SW_Push" (id 1) (at 257.81 53.4924 0))
-    (property "Footprint" "MX_Alps_Hybrid:MXOnly-1U-Hotswap-guide" (id 2) (at 257.81 53.34 0)
+    (property "Footprint" "MX_Alps_Hybrid:MXOnly-1U-NoLED" (id 2) (at 257.81 53.34 0)
       (effects (font (size 1.27 1.27)) hide)
     )
@@
     (property "Reference" "SW_1" (id 0) (at 59.69 51.181 0))
     (property "Value" "SW_Push" (id 1) (at 59.69 53.4924 0))
-    (property "Footprint" "MX_Alps_Hybrid:MXOnly-1U-Hotswap-guide" (id 2) (at 59.69 53.34 0)
+    (property "Footprint" "MX_Alps_Hybrid:MXOnly-1U-NoLED" (id 2) (at 59.69 53.34 0)
       (effects (font (size 1.27 1.27)) hide)
     )
@@
     (property "Reference" "SW_[1" (id 0) (at 142.24 82.931 0))
     (property "Value" "SW_Push" (id 1) (at 142.24 85.2424 0))
-    (property "Footprint" "MX_Alps_Hybrid:MXOnly-1U-Hotswap-guide" (id 2) (at 142.24 85.09 0)
+    (property "Footprint" "MX_Alps_Hybrid:MXOnly-1U-NoLED" (id 2) (at 142.24 85.09 0)
       (effects (font (size 1.27 1.27)) hide)
     )
@@
     (property "Reference" "SW_\\1" (id 0) (at 175.26 51.181 0))
     (property "Value" "SW_Push" (id 1) (at 175.26 53.4924 0))
-    (property "Footprint" "MX_Alps_Hybrid:MXOnly-1U-Hotswap-guide" (id 2) (at 175.26 53.34 0)
-      (effects (font (size 1.27 1.27)) hide)
-    )
+    (property "Footprint" "MX_Alps_Hybrid:MXOnly-1U-NoLED" (id 2) (at 175.26 53.34 0)
+      (effects (font (size 1.27 1.27)) hide)
+    )
