File: PCB/Sandy_Base/Sandy_Base.kicad_sch (KiCad schematic)
At the start: 171 parts, among them J1 USB_C_Receptacle_USB2.0, J10 Conn_02x02_Top_Bottom, J15 Conn_02x02_Top_Bottom, J2 Conn_01x03, J3 Conn_01x02, J4 Conn_02x03_Odd_Even, J6 Conn_02x02_Top_Bottom, J7 Conn_02x02_Top_Bottom, J8 Conn_02x02_Top_Bottom, J9 Conn_02x02_Top_Bottom, U1 ATmega32U4-MU, U2 24LC64, Y1 16MHz

Commit message: LEDに3Dモデルを追加
Parts:
- LED1, LED2, LED3, LED4: footprint locallib:LED_SK6812MINI_PLCC4_3.5x3.5mm_P1.75mm_TriangleMark_Thick -> locallib:LED_SK6812MINI_PLCC4_3.5x3.5mm_P1.75mm_minimal
Changed lines of the file:
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@@
       (effects (font (size 1.27 1.27)) (justify left))
     )
-    (property "Footprint" "locallib:LED_SK6812MINI_PLCC4_3.5x3.5mm_P1.75mm_TriangleMark_Thick" (id 2) (at 307.34 220.98 0)
+    (property "Footprint" "locallib:LED_SK6812MINI_PLCC4_3.5x3.5mm_P1.75mm_minimal" (id 2) (at 307.34 220.98 0)
       (effects (font (size 1.27 1.27)) (justify left top) hide)
     )
@@
       (effects (font (size 1.27 1.27)) (justify left))
     )
-    (property "Footprint" "locallib:LED_SK6812MINI_PLCC4_3.5x3.5mm_P1.75mm_TriangleMark_Thick" (id 2) (at 322.58 220.98 0)
+    (property "Footprint" "locallib:LED_SK6812MINI_PLCC4_3.5x3.5mm_P1.75mm_minimal" (id 2) (at 322.58 220.98 0)
       (effects (font (size 1.27 1.27)) (justify left top) hide)
     )
@@
       (effects (font (size 1.27 1.27)) (justify left))
     )
-    (property "Footprint" "locallib:LED_SK6812MINI_PLCC4_3.5x3.5mm_P1.75mm_TriangleMark_Thick" (id 2) (at 354.965 220.98 0)
+    (property "Footprint" "locallib:LED_SK6812MINI_PLCC4_3.5x3.5mm_P1.75mm_minimal" (id 2) (at 354.965 220.98 0)
       (effects (font (size 1.27 1.27)) (justify left top) hide)
     )
@@
       (effects (font (size 1.27 1.27)) (justify left))
     )
-    (property "Footprint" "locallib:LED_SK6812MINI_PLCC4_3.5x3.5mm_P1.75mm_TriangleMark_Thick" (id 2) (at 370.205 220.98 0)
+    (property "Footprint" "locallib:LED_SK6812MINI_PLCC4_3.5x3.5mm_P1.75mm_minimal" (id 2) (at 370.205 220.98 0)
       (effects (font (size 1.27 1.27)) (justify left top) hide)
     )
@@
     )
     (path "/00000000-0000-0000-0000-00005f7267dd"
-      (reference "LED1") (unit 1) (value "SK6812MINI") (footprint "locallib:LED_SK6812MINI_PLCC4_3.5x3.5mm_P1.75mm_TriangleMark_Thick")
+      (reference "LED1") (unit 1) (value "SK6812MINI") (footprint "locallib:LED_SK6812MINI_PLCC4_3.5x3.5mm_P1.75mm_minimal")
     )
     (path "/00000000-0000-0000-0000-00005f7283a7"
-      (reference "LED2") (unit 1) (value "SK6812MINI") (footprint "locallib:LED_SK6812MINI_PLCC4_3.5x3.5mm_P1.75mm_TriangleMark_Thick")
+      (reference "LED2") (unit 1) (value "SK6812MINI") (footprint "locallib:LED_SK6812MINI_PLCC4_3.5x3.5mm_P1.75mm_minimal")
     )
     (path "/00000000-0000-0000-0000-000063aabb78"
-      (reference "LED3") (unit 1) (value "SK6812MINI") (footprint "locallib:LED_SK6812MINI_PLCC4_3.5x3.5mm_P1.75mm_TriangleMark_Thick")
+      (reference "LED3") (unit 1) (value "SK6812MINI") (footprint "locallib:LED_SK6812MINI_PLCC4_3.5x3.5mm_P1.75mm_minimal")
     )
     (path "/00000000-0000-0000-0000-000063aabb7e"
-      (reference "LED4") (unit 1) (value "SK6812MINI") (footprint "locallib:LED_SK6812MINI_PLCC4_3.5x3.5mm_P1.75mm_TriangleMark_Thick")
+      (reference "LED4") (unit 1) (value "SK6812MINI") (footprint "locallib:LED_SK6812MINI_PLCC4_3.5x3.5mm_P1.75mm_minimal")
     )
     (path "/00000000-0000-0000-0000-000061cf6e0d"

Commit message: マトリクスとキー使用数についてのメモ追記
Other:
- note added: "Max keys = 10 rows * 8 cols = 80 Physical keys = 15 + 14 + 14 + 15 + 13 = 71 5-way nav = 5 Remap/VIA virtual key assign for 2 encoders = 2 * 2 = 4 Balance = 0 (!)"
Changed lines of the file:
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@@
     (effects (font (size 2.54 2.54) (thickness 0.508) bold) (justify left bottom))
+  )
+  (text "Max keys = 10 rows * 8 cols = 80\nPhysical keys = 15 + 14 + 14 + 15 + 13 = 71\n5-way nav = 5\nRemap/VIA virtual key assign for 2 encoders = 2 * 2 = 4\nBalance = 0 (!)"
+    (at 64.77 26.035 0)
+    (effects (font (size 1.27 1.27)) (justify left bottom))
   )
   (global_label "col2" (shape input) (at 99.06 214.63 0) (fields_autoplaced)

Commit message: SHコネクタのパーツ番号を追加
Parts:
- J10, J15, J6, J7, J8, J9: LCSC (none) -> C371510
Changed lines of the file:
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@@
+      (effects (font (size 1.27 1.27)) hide)
+    )
+    (property "LCSC" "C371510" (id 4) (at 137.16 214.63 0)
       (effects (font (size 1.27 1.27)) hide)
     )
@@
     )
     (property "Datasheet" "~" (id 3) (at 187.96 214.63 0)
+      (effects (font (size 1.27 1.27)) hide)
+    )
+    (property "LCSC" "C371510" (id 4) (at 187.96 214.63 0)
       (effects (font (size 1.27 1.27)) hide)
     )
@@
       (effects (font (size 1.27 1.27)) hide)
     )
+    (property "LCSC" "C371510" (id 4) (at 137.795 259.08 0)
+      (effects (font (size 1.27 1.27)) hide)
+    )
     (pin "1")
     (pin "2")
@@
     )
     (property "Datasheet" "~" (id 3) (at 86.995 259.08 0)
+      (effects (font (size 1.27 1.27)) hide)
+    )
+    (property "LCSC" "C371510" (id 4) (at 86.995 259.08 0)
       (effects (font (size 1.27 1.27)) hide)
     )
@@
       (effects (font (size 1.27 1.27)) hide)
     )
+    (property "LCSC" "C371510" (id 4) (at 86.36 214.63 0)
+      (effects (font (size 1.27 1.27)) hide)
+    )
     (pin "1")
     (pin "2")
@@
       (effects (font (size 1.27 1.27)) hide)
     )
+    (property "LCSC" "C371510" (id 4) (at 36.195 259.08 0)
+      (effects (font (size 1.27 1.27)) hide)
+    )

Commit message: WIP, KiCad7
Parts:
- SW_;1, SW_<1, SW_>1, SW_A1, SW_C1, SW_CenterL1u1, SW_CenterL1u2, SW_CenterR1u1, SW_CenterR1u2, SW_D1, SW_DOWN1, SW_E1, SW_F1, SW_Fn1u1, SW_I1, SW_J1, SW_K1, SW_L1, SW_L2-1u1, SW_LSFT1u1, SW_LSFT1u2, SW_M1, SW_N1, SW_O1, SW_S1, SW_UP1, SW_V1, SW_W1, SW_X1, SW_Z1: footprint MX_Alps_Hybrid:MXOnly-1U-NoLED -> MX_Alps_Hybrid:MXOnly-1U-Hotswap-guide
- SW_CAPS1u1, SW_CenterC1u1, SW_RIGHT1: footprint MX_Alps_Hybrid:MXOnly-1U-NoLED -> MX_Alps_Hybrid:MXOnly-1U-Hotswap-on-RE-guide
- SW_CTL1.25u1, SW_ENT1.25u1, SW_LALT1.25u1, SW_LWIN1.25u1, SW_RALT1.25u1, SW_ROPT1.25u1: footprint MX_Alps_Hybrid:MXOnly-1.25U-NoLED -> MX_Alps_Hybrid:MXOnly-1.25U-Hotswap-guide
- SW_CTL1.5u1, SW_ENT1.5u1, SW_LSPC1.5u1, SW_RSPC1.5u1: footprint MX_Alps_Hybrid:MXOnly-1.5U-NoLED -> MX_Alps_Hybrid:MXOnly-1.5U-Hotswap-guide
- SW_LSFT2u1: footprint MX_Alps_Hybrid:MXOnly-2U-NoLED -> MX_Alps_Hybrid:MXOnly-2U-Hotswap-ReversedStabilizers-guide2
- SW_LSPC2u1: footprint MX_Alps_Hybrid:MXOnly-2U-ReversedStabilizers-NoLED -> MX_Alps_Hybrid:MXOnly-2U-Hotswap-ReversedStabilizers-guide2
- SW_RSPC2u1: footprint MX_Alps_Hybrid:MXOnly-2U-ReversedStabilizers-NoLED -> MX_Alps_Hybrid:MXOnly-2U-Hotswap-guide2
- U1: footprint Housings_DFN_QFN:QFN-44-1EP_7x7mm_Pitch0.5mm -> Package_DFN_QFN:QFN-44-1EP_7x7mm_P0.5mm_EP5.2x5.2mm
- renumbered RE_L2 to #RE_L3, RE_R2 to #RE_R2, SW_LSFT1.75u1 to #SW_LSFT1.75u1, RE_L3 to RE_L2

Commit message: WIP
Parts:
- removed JP_LED1, JP_LED2: SolderJumper_3_Open, Jumper:SolderJumper-3_P1.3mm_Open_Pad1.0x1.5mm_NumberLabels, symbol Sandy-rescue:SolderJumper_3_Open-Jumper
- SW_LSPC2u1: footprint MX_Alps_Hybrid:MXOnly-2U-Hotswap-ReversedStabilizers-guide2 -> MX_Alps_Hybrid:MXOnly-2U-Hotswap-guide2
Connections:
- net LED: now also LED1.3 (DIN)
- net at LED2.1 (DOUT): now also LED3.3 (DIN)
Other:
- note added: "Left side"
- note added: "Right side"
- note removed: "Use Left LEDs"
- note removed: "Use Right LEDs"

Commit message: WIP
Parts:
- SW_CenterC1u1: footprint MX_Alps_Hybrid:MXOnly-1U-Hotswap-on-RE-guide -> MX_Alps_Hybrid:MXOnly-1U-Hotswap-custom1-guide
- SW_CenterL1u1, SW_CenterR1u1: footprint MX_Alps_Hybrid:MXOnly-1U-Hotswap-guide -> MX_Alps_Hybrid:MXOnly-1U-Hotswap-custom1-guide
- SW_CenterL1u2: footprint MX_Alps_Hybrid:MXOnly-1U-Hotswap-guide -> MX_Alps_Hybrid:MXOnly-1U-Hotswap-custom2-guide
- SW_CenterR1u2: footprint MX_Alps_Hybrid:MXOnly-1U-Hotswap-guide -> MX_Alps_Hybrid:MXOnly-1U-Hotswap-custom3-guide
Changed lines of the file:
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@@
       (effects (font (size 1.27 1.27)))
     )
-    (property "Footprint" "MX_Alps_Hybrid:MXOnly-1U-Hotswap-guide" (at 128.27 172.72 0)
+    (property "Footprint" "MX_Alps_Hybrid:MXOnly-1U-Hotswap-custom1-guide" (at 128.27 172.72 0)
       (effects (font (size 1.27 1.27)) hide)
     )
@@
       (effects (font (size 1.27 1.27)))
     )
-    (property "Footprint" "MX_Alps_Hybrid:MXOnly-1U-Hotswap-guide" (at 161.29 172.72 0)
+    (property "Footprint" "MX_Alps_Hybrid:MXOnly-1U-Hotswap-custom1-guide" (at 161.29 172.72 0)
       (effects (font (size 1.27 1.27)) hide)
     )
@@
       (effects (font (size 1.27 1.27)))
     )
-    (property "Footprint" "MX_Alps_Hybrid:MXOnly-1U-Hotswap-on-RE-guide" (at 144.78 172.72 0)
+    (property "Footprint" "MX_Alps_Hybrid:MXOnly-1U-Hotswap-custom1-guide" (at 144.78 172.72 0)
       (effects (font (size 1.27 1.27)) hide)
     )
@@
       (effects (font (size 1.27 1.27)))
     )
-    (property "Footprint" "MX_Alps_Hybrid:MXOnly-1U-Hotswap-guide" (at 128.27 167.64 0)
+    (property "Footprint" "MX_Alps_Hybrid:MXOnly-1U-Hotswap-custom2-guide" (at 128.27 167.64 0)
       (effects (font (size 1.27 1.27)) hide)
     )
@@
       (effects (font (size 1.27 1.27)))
     )
-    (property "Footprint" "MX_Alps_Hybrid:MXOnly-1U-Hotswap-guide" (at 161.29 167.64 0)
-      (effects (font (size 1.27 1.27)) hide)
-    )
+    (property "Footprint" "MX_Alps_Hybrid:MXOnly-1U-Hotswap-custom3-guide" (at 161.29 167.64 0)
+      (effects (font (size 1.27 1.27)) hide)
+    )

Commit message: WIP, I2Cの抵抗をネジ穴から離す
Parts:
- SW_CenterC1u1: footprint MX_Alps_Hybrid:MXOnly-1U-Hotswap-custom1-guide -> MX_Alps_Hybrid:MXOnly-1U-Hotswap-custom4-guide
Changed lines of the file:
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@@
       (effects (font (size 1.27 1.27)))
     )
-    (property "Footprint" "MX_Alps_Hybrid:MXOnly-1U-Hotswap-custom1-guide" (at 144.78 172.72 0)
+    (property "Footprint" "MX_Alps_Hybrid:MXOnly-1U-Hotswap-custom4-guide" (at 144.78 172.72 0)
       (effects (font (size 1.27 1.27)) hide)
     )

Commit message: WIP, issue #61
Parts:
- renumbered J6 to J1, J2 to J10, J9 to J2, J10 to J3, J15 to J4, J8 to J5, J7 to J6, J1 to J7, J4 to J8, J3 to J9
Changed lines of the file:
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@@
   (symbol (lib_id "Connector_Generic:Conn_01x03") (at 393.7 213.36 0) (unit 1)
     (in_bom yes) (on_board yes) (dnp no)
-    (property "Reference" "J2" (at 395.732 212.2932 0)
+    (property "Reference" "J10" (at 395.732 212.2932 0)
       (effects (font (size 1.27 1.27)) (justify left))
     )
@@
       (project "Sandy_Base"
         (path "/a99ab643-cdc7-4f8c-8088-c1f4faa914d1"
-          (reference "J2") (unit 1)
+          (reference "J10") (unit 1)
         )
       )
@@
   (symbol (lib_id "Connector_Generic:Conn_02x03_Odd_Even") (at 300.99 41.275 0) (unit 1)
     (in_bom yes) (on_board yes) (dnp no)
-    (property "Reference" "J4" (at 302.26 33.2232 0)
+    (property "Reference" "J8" (at 302.26 33.2232 0)
       (effects (font (size 1.27 1.27)))
     )
@@
       (project "Sandy_Base"
         (path "/a99ab643-cdc7-4f8c-8088-c1f4faa914d1"
-          (reference "J4") (unit 1)
+          (reference "J8") (unit 1)
         )
       )
@@
   (symbol (lib_id "Connector_Generic:Conn_01x02") (at 312.42 114.3 0) (unit 1)
     (in_bom yes) (on_board yes) (dnp no)
-    (property "Reference" "J3" (at 314.452 114.5032 0)
+    (property "Reference" "J9" (at 314.452 114.5032 0)
       (effects (font (size 1.27 1.27)) (justify left))
     )
@@
       (project "Sandy_Base"
         (path "/a99ab643-cdc7-4f8c-8088-c1f4faa914d1"
-          (reference "J3") (unit 1)
+          (reference "J9") (unit 1)
         )
       )
@@
   (symbol (lib_id "Connector:USB_C_Receptacle_USB2.0") (at 330.2 167.64 0) (unit 1)
     (in_bom yes) (on_board yes) (dnp no)
-    (property "Reference" "J1" (at 332.9178 145.6182 0)
+    (property "Reference" "J7" (at 332.9178 145.6182 0)
       (effects (font (size 1.27 1.27)))
     )
@@
       (project "Sandy_Base"
         (path "/a99ab643-cdc7-4f8c-8088-c1f4faa914d1"
-          (reference "J1") (unit 1)
+          (reference "J7") (unit 1)
         )
       )
@@
   (symbol (lib_id "Connector_Generic:Conn_02x02_Odd_Even") (at 137.16 214.63 0) (unit 1)
     (in_bom yes) (on_board yes) (dnp no) (fields_autoplaced)
-    (property "Reference" "J7" (at 138.43 209.6602 0)
-      (effects (font (size 1.27 1.27)))
-    )
-    (property "Value" "Conn_02x02_Top_Bottom" (at 138.43 212.1971 0)
+    (property "Reference" "J6" (at 138.43 210.3501 0)
+      (effects (font (size 1.27 1.27)))
+    )
+    (property "Value" "Conn_02x02_Top_Bottom" (at 138.43 212.2711 0)
       (effects (font (size 1.27 1.27)))
     )
@@
       (project "Sandy_Base"
         (path "/a99ab643-cdc7-4f8c-8088-c1f4faa914d1"
-          (reference "J7") (unit 1)
+          (reference "J6") (unit 1)
         )
       )
@@
   (symbol (lib_id "Connector_Generic:Conn_02x02_Odd_Even") (at 187.96 214.63 0) (unit 1)
     (in_bom yes) (on_board yes) (dnp no) (fields_autoplaced)
-    (property "Reference" "J8" (at 189.23 209.6602 0)
-      (effects (font (size 1.27 1.27)))
-    )
-    (property "Value" "Conn_02x02_Top_Bottom" (at 189.23 212.1971 0)
+    (property "Reference" "J5" (at 189.23 210.3501 0)
+      (effects (font (size 1.27 1.27)))
+    )
+    (property "Value" "Conn_02x02_Top_Bottom" (at 189.23 212.2711 0)
       (effects (font (size 1.27 1.27)))
     )
@@
       (project "Sandy_Base"
         (path "/a99ab643-cdc7-4f8c-8088-c1f4faa914d1"
-          (reference "J8") (unit 1)
+          (reference "J5") (unit 1)
         )
       )
@@
   (symbol (lib_id "Connector_Generic:Conn_02x02_Odd_Even") (at 137.795 259.08 0) (unit 1)
     (in_bom yes) (on_board yes) (dnp no) (fields_autoplaced)
-    (property "Reference" "J15" (at 139.065 254.1102 0)
-      (effects (font (size 1.27 1.27)))
-    )
-    (property "Value" "Conn_02x02_Top_Bottom" (at 139.065 256.6471 0)
+    (property "Reference" "J4" (at 139.065 254.8001 0)
+      (effects (font (size 1.27 1.27)))
+    )
+    (property "Value" "Conn_02x02_Top_Bottom" (at 139.065 256.7211 0)
       (effects (font (size 1.27 1.27)))
     )
@@
       (project "Sandy_Base"
         (path "/a99ab643-cdc7-4f8c-8088-c1f4faa914d1"
-          (reference "J15") (unit 1)
+          (reference "J4") (unit 1)
         )
       )
@@
   (symbol (lib_id "Connector_Generic:Conn_02x02_Odd_Even") (at 86.995 259.08 0) (unit 1)
     (in_bom yes) (on_board yes) (dnp no) (fields_autoplaced)
-    (property "Reference" "J10" (at 88.265 254.1102 0)
-      (effects (font (size 1.27 1.27)))
-    )
-    (property "Value" "Conn_02x02_Top_Bottom" (at 88.265 256.6471 0)
+    (property "Reference" "J3" (at 88.265 254.8001 0)
+      (effects (font (size 1.27 1.27)))
+    )
+    (property "Value" "Conn_02x02_Top_Bottom" (at 88.265 256.7211 0)
       (effects (font (size 1.27 1.27)))
     )
@@
       (project "Sandy_Base"
         (path "/a99ab643-cdc7-4f8c-8088-c1f4faa914d1"
-          (reference "J10") (unit 1)
+          (reference "J3") (unit 1)
         )
       )
@@
   (symbol (lib_id "Connector_Generic:Conn_02x02_Odd_Even") (at 86.36 214.63 0) (unit 1)
     (in_bom yes) (on_board yes) (dnp no) (fields_autoplaced)
-    (property "Reference" "J6" (at 87.63 209.6602 0)
-      (effects (font (size 1.27 1.27)))
-    )
-    (property "Value" "Conn_02x02_Top_Bottom" (at 87.63 212.1971 0)
+    (property "Reference" "J1" (at 87.63 210.3501 0)
+      (effects (font (size 1.27 1.27)))
+    )
+    (property "Value" "Conn_02x02_Top_Bottom" (at 87.63 212.2711 0)
       (effects (font (size 1.27 1.27)))
     )
@@
       (project "Sandy_Base"
         (path "/a99ab643-cdc7-4f8c-8088-c1f4faa914d1"
-          (reference "J6") (unit 1)
+          (reference "J1") (unit 1)
         )
       )
@@
   (symbol (lib_id "Connector_Generic:Conn_02x02_Odd_Even") (at 36.195 259.08 0) (unit 1)
     (in_bom yes) (on_board yes) (dnp no) (fields_autoplaced)
-    (property "Reference" "J9" (at 37.465 254.1102 0)
-      (effects (font (size 1.27 1.27)))
-    )
-    (property "Value" "Conn_02x02_Top_Bottom" (at 37.465 256.6471 0)
+    (property "Reference" "J2" (at 37.465 254.8001 0)
+      (effects (font (size 1.27 1.27)))
+    )
+    (property "Value" "Conn_02x02_Top_Bottom" (at 37.465 256.7211 0)
       (effects (font (size 1.27 1.27)))
     )
@@
       (project "Sandy_Base"
         (path "/a99ab643-cdc7-4f8c-8088-c1f4faa914d1"
-          (reference "J9") (unit 1)
-        )
-      )
+          (reference "J2") (unit 1)
+        )
+      )
