File: PCB/Sandy_Base/Sandy_Base.kicad_sch (KiCad schematic)
At the start: 181 parts, among them J1 Conn_02x02_Top_Bottom, J10 Conn_01x03, J2 Conn_02x02_Top_Bottom, J3 Conn_02x02_Top_Bottom, J4 Conn_02x02_Top_Bottom, J5 Conn_02x02_Top_Bottom, J6 Conn_02x02_Top_Bottom, J7 USB_C_Receptacle_USB2.0, J8 Conn_02x03_Odd_Even, J9 Conn_01x02, U1 ATmega32U4-MU, U2 24LC64, Y1 16MHz

Commit message: WIP:　アンダーグローLED #98
Parts:
- C1: footprint locallib:YS-SK6812MINI-E_middle_hole_with_small_pad -> Capacitor_SMD:C_0805_2012Metric
- C2, C3, C4, C5, C6, C7: footprint Capacitor_SMD:C_0805_2012Metric_Pad1.18x1.45mm_HandSolder -> Capacitor_SMD:C_0805_2012Metric
- R1, R2, R3, R4, R5, R6, R8, R9: footprint Resistor_SMD:R_0805_2012Metric_Pad1.20x1.40mm_HandSolder -> Resistor_SMD:R_0805_2012Metric
Connections:
- no-connect marks 3 -> 4
Changed lines of the file:
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@@
   )
   (no_connect (at 345.44 180.34))
+  (no_connect (at 480.06 208.28))
   (no_connect (at 345.44 182.88))
   (no_connect (at 358.775 57.785))
@@
       (effects (font (size 1.27 1.27)) (justify left))
     )
-    (property "Footprint" "Capacitor_SMD:C_0805_2012Metric_Pad1.18x1.45mm_HandSolder" (at 353.06 75.565 0)
+    (property "Footprint" "Capacitor_SMD:C_0805_2012Metric" (at 353.06 75.565 0)
       (effects (font (size 1.27 1.27)) hide)
     )
@@
       (effects (font (size 1.27 1.27)) (justify left))
     )
-    (property "Footprint" "Resistor_SMD:R_0805_2012Metric_Pad1.20x1.40mm_HandSolder" (at 353.06 36.83 0)
+    (property "Footprint" "Resistor_SMD:R_0805_2012Metric" (at 353.06 36.83 0)
       (effects (font (size 1.27 1.27)) hide)
     )
@@
       (effects (font (size 1.27 1.27)) (justify left))
     )
-    (property "Footprint" "Capacitor_SMD:C_0805_2012Metric_Pad1.18x1.45mm_HandSolder" (at 334.645 47.625 0)
+    (property "Footprint" "Capacitor_SMD:C_0805_2012Metric" (at 334.645 47.625 0)
       (effects (font (size 1.27 1.27)) hide)
     )
@@
       (effects (font (size 1.27 1.27)) (justify left))
     )
-    (property "Footprint" "Capacitor_SMD:C_0805_2012Metric_Pad1.18x1.45mm_HandSolder" (at 334.645 55.245 0)
+    (property "Footprint" "Capacitor_SMD:C_0805_2012Metric" (at 334.645 55.245 0)
       (effects (font (size 1.27 1.27)) hide)
     )
@@
       (effects (font (size 1.27 1.27)) (justify left))
     )
-    (property "Footprint" "Resistor_SMD:R_0805_2012Metric_Pad1.20x1.40mm_HandSolder" (at 398.78 95.885 0)
+    (property "Footprint" "Resistor_SMD:R_0805_2012Metric" (at 398.78 95.885 0)
       (effects (font (size 1.27 1.27)) hide)
     )
@@
       (effects (font (size 1.27 1.27)) (justify left))
     )
-    (property "Footprint" "Capacitor_SMD:C_0805_2012Metric_Pad1.18x1.45mm_HandSolder" (at 339.09 97.79 0)
+    (property "Footprint" "Capacitor_SMD:C_0805_2012Metric" (at 339.09 97.79 0)
       (effects (font (size 1.27 1.27)) hide)
     )
@@
       (effects (font (size 1.27 1.27)) (justify left))
     )
-    (property "Footprint" "Capacitor_SMD:C_0805_2012Metric_Pad1.18x1.45mm_HandSolder" (at 345.44 97.79 0)
+    (property "Footprint" "Capacitor_SMD:C_0805_2012Metric" (at 345.44 97.79 0)
       (effects (font (size 1.27 1.27)) hide)
     )
@@
       (effects (font (size 1.27 1.27)) (justify left))
     )
-    (property "Footprint" "Capacitor_SMD:C_0805_2012Metric_Pad1.18x1.45mm_HandSolder" (at 351.79 97.79 0)
+    (property "Footprint" "Capacitor_SMD:C_0805_2012Metric" (at 351.79 97.79 0)
       (effects (font (size 1.27 1.27)) hide)
     )
@@
       (effects (font (size 1.27 1.27)) (justify left))
     )
-    (property "Footprint" "locallib:YS-SK6812MINI-E_middle_hole_with_small_pad" (at 332.74 97.79 0)
+    (property "Footprint" "Capacitor_SMD:C_0805_2012Metric" (at 332.74 97.79 0)
       (effects (font (size 1.27 1.27)) hide)
     )
@@
       (effects (font (size 1.27 1.27)) (justify left))
     )
-    (property "Footprint" "Resistor_SMD:R_0805_2012Metric_Pad1.20x1.40mm_HandSolder" (at 375.92 165.1 0)
+    (property "Footprint" "Resistor_SMD:R_0805_2012Metric" (at 375.92 165.1 0)
       (effects (font (size 1.27 1.27)) hide)
     )
@@
       (effects (font (size 1.27 1.27)) (justify left))
     )
-    (property "Footprint" "Resistor_SMD:R_0805_2012Metric_Pad1.20x1.40mm_HandSolder" (at 375.92 170.18 0)
+    (property "Footprint" "Resistor_SMD:R_0805_2012Metric" (at 375.92 170.18 0)
       (effects (font (size 1.27 1.27)) hide)
     )
@@
       (effects (font (size 1.27 1.27)))
     )
-    (property "Footprint" "Resistor_SMD:R_0805_2012Metric_Pad1.20x1.40mm_HandSolder" (at 354.33 160.02 0)
+    (property "Footprint" "Resistor_SMD:R_0805_2012Metric" (at 354.33 160.02 0)
       (effects (font (size 1.27 1.27)) hide)
     )
@@
       (effects (font (size 1.27 1.27)))
     )
-    (property "Footprint" "Resistor_SMD:R_0805_2012Metric_Pad1.20x1.40mm_HandSolder" (at 359.41 157.48 0)
+    (property "Footprint" "Resistor_SMD:R_0805_2012Metric" (at 359.41 157.48 0)
       (effects (font (size 1.27 1.27)) hide)
     )
@@
       (effects (font (size 1.27 1.27)) (justify left))
     )
-    (property "Footprint" "Resistor_SMD:R_0805_2012Metric_Pad1.20x1.40mm_HandSolder" (at 294.132 107.95 90)
+    (property "Footprint" "Resistor_SMD:R_0805_2012Metric" (at 294.132 107.95 90)
       (effects (font (size 1.27 1.27)) hide)
     )
@@
       (effects (font (size 1.27 1.27)) (justify left))
     )
-    (property "Footprint" "Resistor_SMD:R_0805_2012Metric_Pad1.20x1.40mm_HandSolder" (at 302.387 107.95 90)
+    (property "Footprint" "Resistor_SMD:R_0805_2012Metric" (at 302.387 107.95 90)
       (effects (font (size 1.27 1.27)) hide)
     )
