File: PCB/Sandy_Base/Sandy_Base.kicad_pcb (KiCad board)
At the start: 2 copper layers, 285 x 95.1 mm, 173 parts, among them J1 Conn_02x02_Top_Bottom, J11 Conn_02x02_Odd_Even, J2 Conn_02x02_Top_Bottom, J3 Conn_02x02_Top_Bottom, J4 Conn_02x02_Top_Bottom, J5 Conn_02x02_Top_Bottom, J6 Conn_02x02_Top_Bottom, J7 USB_C_Receptacle_USB2.0, J8 Conn_01x03, J9 Conn_01x08_Pin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

Commit message: WIP 配線中
Parts:
- moved J2 0.20 mm to (149.7, 53.0)
- moved J1 0.11 mm to (142.5, 43.8)
- moved J6 0.08 mm to (175.8, 32.9)
Routing:
- net Net-(L2-DOUT): track 0.00 -> 284.4 mm
- net col0: track 210.2 -> 340.7 mm, vias 5 -> 7
- net col1: track 198.5 -> 284.4 mm, vias 5 -> 6
- net col6: track 421.1 -> 456.6 mm
- net Net-(L1-DOUT): track 0.00 -> 11.8 mm
- net Net-(L3-DOUT): track 0.00 -> 10.3 mm
- net GND: track 21.3 -> 24.1 mm
- net RE_Base1_A: track 149.8 -> 147.7 mm
- net +5V: track 342.6 -> 344.2 mm, vias 3 -> 4
- net Audio2: track 248.2 -> 249.4 mm
- net RE_Base1_B: track 143.9 -> 144.9 mm
- net col4: track 297.4 -> 298.0 mm

Commit message: 配線調整
Parts:
- moved C103 1.25 mm to (287.9, 78.5)
- moved C102 1.20 mm to (25.9, 85.6)
- moved C104 1.20 mm to (287.9, 85.6)
- moved C101 1.20 mm to (25.9, 78.5)
- moved L1 1.19 mm to (28.2, 80.6)
- moved L2 1.19 mm to (28.2, 87.7)
- moved L3 1.19 mm to (290.1, 80.6)
- moved L4 1.19 mm to (290.1, 87.7)
Routing:
- net row7: track 320.7 -> 324.3 mm
- net Net-(L1-DOUT): track 11.8 -> 8.69 mm
- net Net-(L3-DOUT): track 10.3 -> 8.75 mm
- net LED_D_5V: track 37.4 -> 38.6 mm
- net +5V: track 344.2 -> 343.4 mm
- net GND: vias 3 -> 7

Commit message: 配線調整
Parts:
- J7: footprint Connector_USB:USB_C_Receptacle_HRO_TYPE-C-31-M-12 -> locallib:USB_C_Receptacle_HRO_TYPE-C-31-M-12
Routing:
- net row3: track 340.0 -> 342.8 mm
- net col6: track 456.6 -> 459.0 mm
- net row0: track 353.4 -> 351.6 mm
- net row9: track 287.6 -> 289.2 mm
- net row6: track 302.9 -> 304.3 mm
- net row8: track 352.5 -> 351.2 mm
- net row2: track 324.1 -> 325.2 mm
- net col4: track 298.0 -> 297.2 mm
- net RESET: track 42.1 -> 41.4 mm
- net row5: track 281.8 -> 281.2 mm
- net row7: track 324.3 -> 323.7 mm
- net GND: vias 7 -> 8

Commit message: USB配線長調整
Routing:
- net D-: track 18.5 -> 19.4 mm
