File: PCB/Sandy_Base/Sandy_Base.kicad_pcb (KiCad board)
At the start: 2 copper layers, 285 x 95.1 mm, 173 parts, among them J1 Conn_02x02_Top_Bottom, J11 Conn_02x02_Odd_Even, J2 Conn_02x02_Top_Bottom, J3 Conn_02x02_Top_Bottom, J4 Conn_02x02_Top_Bottom, J5 Conn_02x02_Top_Bottom, J6 Conn_02x02_Top_Bottom, J7 USB_C_Receptacle_USB2.0, J8 Conn_01x03, J9 Conn_01x08_Pin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

Commit message: 配線調整
Parts:
- J8: footprint Connector_PinHeader_2.54mm:PinHeader_1x03_P2.54mm_Vertical -> locallib:PinHeader_1x03_P2.54mm_Vertical_All_circle
- J9: footprint Connector_PinHeader_1.00mm:PinHeader_1x08_P1.00mm_Vertical -> locallib:PinHeader_1x08_P1.00mm_Vertical_All_circle
Routing:
- net col3: track 217.7 -> 206.7 mm
- net col6: track 459.0 -> 455.5 mm
- net col1: track 284.4 -> 286.8 mm
- net GND: track 24.1 -> 26.1 mm
- net row6: track 304.3 -> 302.9 mm, vias 2 -> 3
- net row0: track 351.6 -> 352.3 mm
- net col5: track 393.2 -> 393.9 mm

Commit message: 配線調整
Routing:
- net col4: track 297.5 -> 294.7 mm
- net col6: track 455.5 -> 453.0 mm
- net GND: track 26.1 -> 24.1 mm, vias 8 -> 11
- net col3: track 206.7 -> 208.6 mm, vias 3 -> 2
- net row8: track 351.2 -> 350.1 mm
- net row0: track 352.3 -> 353.4 mm
- net row3: track 342.8 -> 341.9 mm
- net row2: track 325.1 -> 324.6 mm

Commit message: USB配線長調整
Parts:
- moved J11 3.80 mm to (32.5, 68.7)
Routing:
- net RESET: track 41.4 -> 45.2 mm
- net USB_BOOT: track 59.4 -> 63.2 mm
- net +5V: track 343.4 -> 345.4 mm
- net D-: track 19.4 -> 18.4 mm
- net row2: track 324.6 -> 325.4 mm
- net D+: track 19.8 -> 19.1 mm

Commit message: ベタにGND打ち
Parts:
- moved G*** 1.50 mm to (159.2, 67.2)
Routing:
- net col3: track 208.6 -> 204.7 mm, vias 2 -> 3
- net row2: track 325.4 -> 324.2 mm
- net row1: track 296.6 -> 295.9 mm
- net col0: track 341.1 -> 341.6 mm
- net GND: vias 11 -> 188
