File: PCB/Sandy_Plate_Top/Sandy_Plate_Top.kicad_pcb (KiCad board)
At the start: 2 copper layers, 285 x 37 mm, 21 parts

Commit message: バージョン表記調整
Other:
- board text added: "#Sandy_kbd v.0.2, Plate for Top by @jpskenn"
- board text removed: "#Sandy_kbd v.0.2, Top plate by @jpskenn"
Changed lines of the file:
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@@
     (fp_arc (start 140.35 -3.025) (mid 140.203553 -2.671447) (end 139.85 -2.525)
       (stroke (width 0.15) (type solid)) (layer "Edge.Cuts"))
-    (fp_arc (start 140.475 -18.75004) (mid 141.889222 -18.164279) (end 142.475 -16.75004)
+    (fp_arc (start 140.475 -18.75004) (mid 141.889257 -18.164285) (end 142.475 -16.75004)
       (stroke (width 0.3) (type solid)) (layer "Edge.Cuts"))
-    (fp_arc (start 142.475 -2.814254) (mid 141.889197 -1.40007) (end 140.475 -0.814254)
+    (fp_arc (start 142.475 -2.814254) (mid 141.889203 -1.400035) (end 140.475 -0.814254)
       (stroke (width 0.3) (type solid)) (layer "Edge.Cuts"))
     (group "" (id b45a4e6d-43e9-43f3-99a8-109a97b956a9)
@@
     (effects (font (size 1.5 1.5) (thickness 0.3)) (justify mirror))
   )
-  (gr_text "#Sandy_kbd v.0.2, Top plate\nby @jpskenn" (at 170.3 36.5) (layer "B.SilkS")
-    (effects (font (size 1.5 1.5) (thickness 0.15)) (justify left mirror))
+  (gr_text "#Sandy_kbd v.0.2, Plate for Top by @jpskenn" (at 193.69906 36.528405) (layer "B.SilkS")
+    (effects (font (size 1.6 1.6) (thickness 0.2)) (justify left mirror))
   )
   (dimension locked (type aligned) (layer "Dwgs.User")

Commit message: ERC, DRCチェック
Changed lines of the file:
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@@
     (fp_arc (start 140.35 -3.025) (mid 140.203553 -2.671447) (end 139.85 -2.525)
       (stroke (width 0.15) (type solid)) (layer "Edge.Cuts"))
-    (fp_arc (start 140.475 -18.75004) (mid 141.889257 -18.164285) (end 142.475 -16.75004)
+    (fp_arc (start 140.475 -18.75004) (mid 141.889222 -18.164279) (end 142.475 -16.75004)
       (stroke (width 0.3) (type solid)) (layer "Edge.Cuts"))
-    (fp_arc (start 142.475 -2.814254) (mid 141.889203 -1.400035) (end 140.475 -0.814254)
+    (fp_arc (start 142.475 -2.814254) (mid 141.889197 -1.40007) (end 140.475 -0.814254)
       (stroke (width 0.3) (type solid)) (layer "Edge.Cuts"))
     (group "" (id b45a4e6d-43e9-43f3-99a8-109a97b956a9)
