File: PCB/Sandy_Plate_Top/Sandy_Plate_Top.kicad_sch (KiCad schematic)
At the start: 19 parts

Commit message: Topプレート
Parts:
- SW_-1, SW_1, SW_10, SW_2, SW_3, SW_4, SW_5, SW_6, SW_7, SW_8, SW_9, SW_=1, SW_ESC1, SW_T1, SW_Y1, SW_[1, SW_\1, SW_]1, SW_`1: footprint MX_Alps_Hybrid:MX-1U-cutout -> Jones.local:MXOnly-1U-Hotswap-guide-dummy
Changed lines of the file:
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@@
       (effects (font (size 1.27 1.27)))
     )
-    (property "Footprint" "MX_Alps_Hybrid:MX-1U-cutout" (at 44.45 43.815 0)
+    (property "Footprint" "Jones.local:MXOnly-1U-Hotswap-guide-dummy" (at 44.45 43.815 0)
       (effects (font (size 1.27 1.27)) hide)
     )
@@
       (effects (font (size 1.27 1.27)))
     )
-    (property "Footprint" "MX_Alps_Hybrid:MX-1U-cutout" (at 193.04 43.815 0)
+    (property "Footprint" "Jones.local:MXOnly-1U-Hotswap-guide-dummy" (at 193.04 43.815 0)
       (effects (font (size 1.27 1.27)) hide)
     )
@@
       (effects (font (size 1.27 1.27)))
     )
-    (property "Footprint" "MX_Alps_Hybrid:MX-1U-cutout" (at 77.47 43.815 0)
+    (property "Footprint" "Jones.local:MXOnly-1U-Hotswap-guide-dummy" (at 77.47 43.815 0)
       (effects (font (size 1.27 1.27)) hide)
     )
@@
       (effects (font (size 1.27 1.27)))
     )
-    (property "Footprint" "MX_Alps_Hybrid:MX-1U-cutout" (at 143.51 43.815 0)
+    (property "Footprint" "Jones.local:MXOnly-1U-Hotswap-guide-dummy" (at 143.51 43.815 0)
       (effects (font (size 1.27 1.27)) hide)
     )
@@
       (effects (font (size 1.27 1.27)))
     )
-    (property "Footprint" "MX_Alps_Hybrid:MX-1U-cutout" (at 127 75.565 0)
+    (property "Footprint" "Jones.local:MXOnly-1U-Hotswap-guide-dummy" (at 127 75.565 0)
       (effects (font (size 1.27 1.27)) hide)
     )
@@
       (effects (font (size 1.27 1.27)))
     )
-    (property "Footprint" "MX_Alps_Hybrid:MX-1U-cutout" (at 160.02 43.815 0)
+    (property "Footprint" "Jones.local:MXOnly-1U-Hotswap-guide-dummy" (at 160.02 43.815 0)
       (effects (font (size 1.27 1.27)) hide)
     )
@@
       (effects (font (size 1.27 1.27)))
     )
-    (property "Footprint" "MX_Alps_Hybrid:MX-1U-cutout" (at 259.08 43.815 0)
+    (property "Footprint" "Jones.local:MXOnly-1U-Hotswap-guide-dummy" (at 259.08 43.815 0)
       (effects (font (size 1.27 1.27)) hide)
     )
@@
       (effects (font (size 1.27 1.27)))
     )
-    (property "Footprint" "MX_Alps_Hybrid:MX-1U-cutout" (at 209.55 43.815 0)
+    (property "Footprint" "Jones.local:MXOnly-1U-Hotswap-guide-dummy" (at 209.55 43.815 0)
       (effects (font (size 1.27 1.27)) hide)
     )
@@
       (effects (font (size 1.27 1.27)))
     )
-    (property "Footprint" "MX_Alps_Hybrid:MX-1U-cutout" (at 60.96 43.815 0)
+    (property "Footprint" "Jones.local:MXOnly-1U-Hotswap-guide-dummy" (at 60.96 43.815 0)
       (effects (font (size 1.27 1.27)) hide)
     )
@@
       (effects (font (size 1.27 1.27)))
     )
-    (property "Footprint" "MX_Alps_Hybrid:MX-1U-cutout" (at 127 43.815 0)
+    (property "Footprint" "Jones.local:MXOnly-1U-Hotswap-guide-dummy" (at 127 43.815 0)
       (effects (font (size 1.27 1.27)) hide)
     )
@@
       (effects (font (size 1.27 1.27)))
     )
-    (property "Footprint" "MX_Alps_Hybrid:MX-1U-cutout" (at 226.06 43.815 0)
+    (property "Footprint" "Jones.local:MXOnly-1U-Hotswap-guide-dummy" (at 226.06 43.815 0)
       (effects (font (size 1.27 1.27)) hide)
     )
@@
       (effects (font (size 1.27 1.27)))
     )
-    (property "Footprint" "MX_Alps_Hybrid:MX-1U-cutout" (at 176.53 75.565 0)
+    (property "Footprint" "Jones.local:MXOnly-1U-Hotswap-guide-dummy" (at 176.53 75.565 0)
       (effects (font (size 1.27 1.27)) hide)
     )
@@
       (effects (font (size 1.27 1.27)))
     )
-    (property "Footprint" "MX_Alps_Hybrid:MX-1U-cutout" (at 143.51 75.565 0)
+    (property "Footprint" "Jones.local:MXOnly-1U-Hotswap-guide-dummy" (at 143.51 75.565 0)
       (effects (font (size 1.27 1.27)) hide)
     )
@@
       (effects (font (size 1.27 1.27)))
     )
-    (property "Footprint" "MX_Alps_Hybrid:MX-1U-cutout" (at 242.57 43.815 0)
+    (property "Footprint" "Jones.local:MXOnly-1U-Hotswap-guide-dummy" (at 242.57 43.815 0)
       (effects (font (size 1.27 1.27)) hide)
     )
@@
       (effects (font (size 1.27 1.27)))
     )
-    (property "Footprint" "MX_Alps_Hybrid:MX-1U-cutout" (at 93.98 43.815 0)
+    (property "Footprint" "Jones.local:MXOnly-1U-Hotswap-guide-dummy" (at 93.98 43.815 0)
       (effects (font (size 1.27 1.27)) hide)
     )
@@
       (effects (font (size 1.27 1.27)))
     )
-    (property "Footprint" "MX_Alps_Hybrid:MX-1U-cutout" (at 275.59 43.815 0)
+    (property "Footprint" "Jones.local:MXOnly-1U-Hotswap-guide-dummy" (at 275.59 43.815 0)
       (effects (font (size 1.27 1.27)) hide)
     )
@@
       (effects (font (size 1.27 1.27)))
     )
-    (property "Footprint" "MX_Alps_Hybrid:MX-1U-cutout" (at 160.02 75.565 0)
+    (property "Footprint" "Jones.local:MXOnly-1U-Hotswap-guide-dummy" (at 160.02 75.565 0)
       (effects (font (size 1.27 1.27)) hide)
     )
@@
       (effects (font (size 1.27 1.27)))
     )
-    (property "Footprint" "MX_Alps_Hybrid:MX-1U-cutout" (at 110.49 43.815 0)
+    (property "Footprint" "Jones.local:MXOnly-1U-Hotswap-guide-dummy" (at 110.49 43.815 0)
       (effects (font (size 1.27 1.27)) hide)
     )
@@
       (effects (font (size 1.27 1.27)))
     )
-    (property "Footprint" "MX_Alps_Hybrid:MX-1U-cutout" (at 176.53 43.815 0)
-      (effects (font (size 1.27 1.27)) hide)
-    )
+    (property "Footprint" "Jones.local:MXOnly-1U-Hotswap-guide-dummy" (at 176.53 43.815 0)
+      (effects (font (size 1.27 1.27)) hide)
+    )

Commit message: Top用プレート作成（穴はEdge.Cutじゃない方法で）
Parts:
- removed SW_=1: SW_Push, Jones.local:MXOnly-1U-Hotswap-guide-dummy, symbol Switch:SW_Push
- added SW_'1, SW_;1: SW_Push, Jones.local:MXOnly-1U-Hotswap-guide-dummy, symbol Switch:SW_Push
- renumbered SW_6 to SW_-1, SW_\1 to SW_6, SW_`1 to SW_=1, SW_-1 to SW_INS1
Connections:
- net Top_col3: now also SW_;1.1
- net Top_col4: now also SW_'1.1
