File: PCB/Sandy_Plate_Bottom/Sandy_Plate_Bottom.kicad_pcb (KiCad board)
At the start: 2 copper layers, 285 x 94.6 mm, 10 parts

Commit message: 更新：ビルドナンバー　→　DN0030
Other:
- board text added: "Universal 60% Bottom Plate v.1.3.2 by @jpskenn"
- board text removed: "Universal 60% Bottom Plate v.1.3.1 by @jpskenn"
Changed lines of the file:
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@@
   (gr_circle (center 40.62 44.97) (end 42.65 46.1)
     (stroke (width 0.15) (type solid)) (fill none) (layer "Eco1.User"))
-  (gr_text "Universal 60% Bottom Plate v.1.3.1\nby @jpskenn" (at 70.246875 66.675) (layer "F.SilkS")
+  (gr_text "Universal 60% Bottom Plate v.1.3.2\nby @jpskenn" (at 70.246875 66.675) (layer "F.SilkS")
     (effects (font (size 1.8 1.8) (thickness 0.24)) (justify left))
   )

Commit message: 変更：ボトムプレート裏側のデザイン性向上
Parts:
- added G***: LOGO, locallib:Sandy_logo_w253, B.Cu at (157.9, 64.0)

Commit message: ファイル名からアスタリスクを削除
Parts:
- G***: footprint locallib:Nora_logo_21.8*7.7 -> locallib:Nora_logo_21.8x7.7
Changed lines of the file:
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@@
     (pad "" np_thru_hole circle (at 0 0) (size 2.2 2.2) (drill 2.2) (layers "*.Cu" "*.Mask"))
   )
-  (footprint "locallib:Nora_logo_21.8*7.7" (layer "F.Cu")
+  (footprint "locallib:Nora_logo_21.8x7.7" (layer "F.Cu")
     (at 207.16875 67.5)
     (attr board_only exclude_from_pos_files exclude_from_bom)

Commit message: ネジ穴調整、追加
Parts:
- removed the G*** at (207.2, 67.5)
- removed the G*** at (171.4, 67.0)
- removed H3, H4, H5: MountingHole, MountingHole:MountingHole_2.2mm_M2
- added H2: MountingHole, MountingHole:MountingHole_2.2mm_M2, F.Cu at (107.9, 106.9)
- added H2: MountingHole, MountingHole:MountingHole_2.2mm_M2, F.Cu at (19.8, 106.9)
- added H2: MountingHole, MountingHole:MountingHole_2.2mm_M2, F.Cu at (296.1, 106.9)
- added H2: MountingHole, MountingHole:MountingHole_2.2mm_M2, F.Cu at (177.0, 21.3)
- added H2: MountingHole, MountingHole:MountingHole_2.2mm_M2, F.Cu at (253.2, 21.3)
- added H2: MountingHole, MountingHole:MountingHole_2.2mm_M2, F.Cu at (208.0, 106.9)
- REF**: footprint locallib:60_Outline_Sandy_Bottom -> locallib:60_Outline_Sandy_DN0040_Bottom
- moved H2 66.7 mm to (138.9, 21.3)
- moved H1 47.6 mm to (62.7, 21.3)
- moved G*** 37.3 mm to (208.0, 66.7)
Other:
- board text added: "Universal 60% Bottom Plate v.1.4.0 by @jpskenn"
- board text removed: "Universal 60% Bottom Plate v.1.3.2 by @jpskenn"

Commit message: Base→Bottomのネジ穴位置変更
Parts:
- added REF**: 1U, locallib:MXOnly-1U-Hotswap-guide-dummy, F.Cu at (281.8, 26.3)
- added REF**: 1U, locallib:MXOnly-1U-Hotswap-guide-dummy, F.Cu at (72.2, 26.3)
- added REF**: 1U, locallib:MXOnly-1U-Hotswap-guide-dummy, F.Cu at (53.2, 26.3)
- added REF**: 1U, locallib:MXOnly-1U-Hotswap-guide-dummy, F.Cu at (148.4, 26.3)
- added REF**: 1U, locallib:MXOnly-1U-Hotswap-guide-dummy, F.Cu at (205.6, 26.3)
- added REF**: 1U, locallib:MXOnly-1U-Hotswap-guide-dummy, F.Cu at (91.3, 26.3)
- added REF**: 1U, locallib:MXOnly-1U-Hotswap-guide-dummy, F.Cu at (34.1, 26.3)
- added REF**: 1U, locallib:MXOnly-1U-Hotswap-guide-dummy, F.Cu at (43.6, 83.5)
- added REF**: 1U, locallib:MXOnly-1U-Hotswap-guide-dummy, F.Cu at (262.7, 26.3)
- added REF**: 1U, locallib:MXOnly-1U-Hotswap-guide-dummy, F.Cu at (129.4, 26.3)
- added REF**: 1U, locallib:MXOnly-1U-Hotswap-guide-dummy, F.Cu at (272.2, 83.5)
- added REF**: 1U, locallib:MXOnly-1U-Hotswap-guide-dummy, F.Cu at (34.1, 45.4)
- added REF**: 1U, locallib:MXOnly-1U-Hotswap-guide-dummy, F.Cu at (167.5, 26.3)
- added REF**: 1U, locallib:MXOnly-1U-Hotswap-guide-dummy, F.Cu at (281.8, 45.4)
- added REF**: 1U, locallib:MXOnly-1U-Hotswap-guide-dummy, F.Cu at (243.7, 26.3)
- added REF**: 1U, locallib:MXOnly-1U-Hotswap-guide-dummy, F.Cu at (34.1, 64.4)
- added REF**: 1U, locallib:MXOnly-1U-Hotswap-guide-dummy, F.Cu at (281.8, 64.4)
- added REF**: 1U, locallib:MXOnly-1U-Hotswap-guide-dummy, F.Cu at (224.6, 26.3)
- added REF**: 1U, locallib:MXOnly-1U-Hotswap-guide-dummy, F.Cu at (186.5, 26.3)
- added REF**: 1U, locallib:MXOnly-1U-Hotswap-guide-dummy, F.Cu at (110.3, 26.3)
- moved H2 21.7 mm to (281.8, 90.6)
- moved H2 21.7 mm to (34.1, 90.6)

Commit message: Base用プレートにネジ穴が見えないよう、ボトムプレートへのネジ位置を調整。
Parts:
- moved H2 19.2 mm to (53.2, 88.2)
- moved H2 19.2 mm to (262.7, 88.2)
Changed lines of the file:
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@@
 	(footprint "MountingHole:MountingHole_2.2mm_M2"
 		(layer "F.Cu")
-		(at 34.125 90.59379)
+		(at 53.175 88.21254)
 		(descr "Mounting Hole 2.2mm, no annular, M2")
 		(tags "mounting hole 2.2mm no annular m2")
@@
 	(footprint "MountingHole:MountingHole_2.2mm_M2"
 		(layer "F.Cu")
-		(at 281.775 90.59379)
+		(at 262.725 88.21254)
 		(descr "Mounting Hole 2.2mm, no annular, M2")
 		(tags "mounting hole 2.2mm no annular m2")
