File: PCB/Sandy_Top/Sandy_Top.kicad_sch (KiCad schematic)
At the start: 45 parts, among them J2 Conn_02x02_Top_Bottom, J3 Conn_02x02_Top_Bottom

Commit message: WIP ネジ位置等検討中
Parts:
- removed H1, H13, H4, H5, H7: MountingHole, locallib:MountingHole_2.2mm_M2_Pad_minimal, symbol Mechanical:MountingHole_Pad
- SW_'1, SW_;1, SW_T1, SW_Y1, SW_[1, SW_]1: footprint MX_Alps_Hybrid:MXOnly-1U-Hotswap-guide -> locallib:Kailh_socket_ChocV2
Connections:
- no-connect marks 5 -> 0
